File: Hardware/Design Files/rfsom-01/emmc.kicad_sch (KiCad schematic)
At the start: 0 parts

Commit message: ddr progress; added more conns;
Parts:
- added C?: CL05B104KA5NNNC, Capacitor_SMD:C_0402_1005Metric_Pad0.74x0.62mm_HandSolder, symbol Capacitors:CL05B104KA5NNNC
- added U?: TXS02612RTWR, ICs:QFN-24-1EP_4x4mm_P0.5mm, symbol ICs:TXS02612RTWR
Connections:
- new net +VCC_1V8: C?.1, U?.5 (VCCA)
- new net +VCC_3V3: U?.17 (VCC_B1), U?.21 (VCC_B0)
- new net GND: C?.2
- new net SD_CLK: U?.9 (CLKA)
- new net SD_CMD: U?.4 (CMDA)
- new net SD_D0: U?.6 (DAT0A)
- new net SD_D1: U?.7 (DAT1A)
- new net SD_D2: U?.1 (DAT2A)
- new net SD_D3: U?.3 (DAT3A)

Commit message: ps progress; added ftdi; mezz pinout pedinging;
Parts:
- removed C?: CL05B104KA5NNNC, Capacitor_SMD:C_0402_1005Metric_Pad0.74x0.62mm_HandSolder, symbol Capacitors:CL05B104KA5NNNC
- removed U?: TXS02612RTWR, ICs:QFN-24-1EP_4x4mm_P0.5mm, symbol ICs:TXS02612RTWR
