File: Hardware/Design Files/rfsom-01/ram.kicad_sch (KiCad schematic)
At the start: 0 parts

Commit message: ddr progress; added more conns;
Parts:
- added C? (x4): CL05B103KB5NNNC, Capacitor_SMD:C_0402_1005Metric, symbol Capacitors:CL05B103KB5NNNC
- added R? (x24): RT0402FRE0740R2L, Resistor_SMD:R_0402_1005Metric, symbol Resistors:RT0402FRE0740R2L
- added R? (x2): RC0402FR-07240RL, Resistor_SMD:R_0402_1005Metric, symbol Resistors:RC0402FR-07240RL
- added U? (x2): AS4C256M16D3C-12BCN, Package_BGA:BGA-96_9.0x13.0mm_Layout2x3x16_P0.8mm, symbol Memory_RAM:AS4C256M16D3
Connections:
- new net: R?.1, U?.L8 (ZQ) (x2)
- new net +VCC_1V5: C?.1, C?.1, U?.A1 (VDDQ), U?.A1 (VDDQ), U?.A8 (VDDQ), U?.A8 (VDDQ), U?.B2 (VDD), U?.B2 (VDD), U?.C1 (VDDQ), U?.C1 (VDDQ), U?.C9 (VDDQ), U?.C9 (VDDQ), U?.D2 (VDDQ), U?.D2 (VDDQ), U?.D9 (VDD), U?.D9 (VDD), U?.E9 (VDDQ), U?.E9 (VDDQ), U?.F1 (VDDQ), U?.F1 (VDDQ), U?.G7 (VDD), U?.G7 (VDD), U?.H2 (VDDQ), U?.H2 (VDDQ), U?.H9 (VDDQ), U?.H9 (VDDQ), U?.K2 (VDD), U?.K2 (VDD), U?.K8 (VDD), U?.K8 (VDD), U?.N1 (VDD), U?.N1 (VDD), U?.N9 (VDD), U?.N9 (VDD), U?.R1 (VDD), U?.R1 (VDD), U?.R9 (VDD), U?.R9 (VDD)
- new net +VTT_0V75: C?.1, C?.1, R?.1, R?.1, R?.1, R?.1, R?.1, R?.1, R?.1, R?.1, R?.1, R?.1, R?.1, R?.1, R?.1, R?.1, R?.1, R?.1, R?.1, R?.1, R?.1, R?.1, R?.1, R?.1, R?.1, R?.1, U?.H1 (VREFDQ), U?.H1 (VREFDQ), U?.M8 (VREFCA), U?.M8 (VREFCA)
- new net DDR3_A0: R?.2
- new net DDR3_A1: R?.2
- new net DDR3_A10: R?.2
- new net DDR3_A11: R?.2
- new net DDR3_A12: R?.2
- new net DDR3_A13: R?.2
- new net DDR3_A14: R?.2
- new net DDR3_A2: R?.2
- new net DDR3_A3: R?.2
- new net DDR3_A4: R?.2
- new net DDR3_A5: R?.2
- new net DDR3_A6: R?.2
- new net DDR3_A7: R?.2
- new net DDR3_A8: R?.2
- new net DDR3_A9: R?.2
- new net DDRA_DM0: U?.E7 (LDM)
- new net DDRA_DM1: U?.D3 (UDM)
- new net DDRA_DQ0: U?.E3 (DQ0)
- new net DDRA_DQ1: U?.F7 (DQ1)
- new net DDRA_DQ10: U?.C8 (DQ10)
- new net DDRA_DQ11: U?.C2 (DQ11)
- new net DDRA_DQ12: U?.A7 (DQ12)
- new net DDRA_DQ13: U?.A2 (DQ13)
- new net DDRA_DQ14: U?.B8 (DQ14)
- new net DDRA_DQ15: U?.A3 (DQ15)
- new net DDRA_DQ2: U?.F2 (DQ2)
- new net DDRA_DQ3: U?.F8 (DQ3)
- new net DDRA_DQ4: U?.H3 (DQ4)
- new net DDRA_DQ5: U?.H8 (DQ5)
- new net DDRA_DQ6: U?.G2 (DQ6)
- new net DDRA_DQ7: U?.H7 (DQ7)
- new net DDRA_DQ8: U?.D7 (DQ8)
- new net DDRA_DQ9: U?.C3 (DQ9)
- new net DDRA_DQS0+: U?.F3 (LDQS)
- new net DDRA_DQS0-: U?.G3 (~{LDQS})
- new net DDRA_DQS1+: U?.C7 (UDQS)
- new net DDRA_DQS1-: U?.B7 (~{UDQS})
- new net DDRB_DM0: U?.E7 (LDM)
- new net DDRB_DM1: U?.D3 (UDM)
- new net DDRB_DQ0: U?.E3 (DQ0)
- new net DDRB_DQ1: U?.F7 (DQ1)
- new net DDRB_DQ10: U?.C8 (DQ10)
- new net DDRB_DQ11: U?.C2 (DQ11)
- new net DDRB_DQ12: U?.A7 (DQ12)
- new net DDRB_DQ13: U?.A2 (DQ13)
- new net DDRB_DQ14: U?.B8 (DQ14)
- new net DDRB_DQ15: U?.A3 (DQ15)
- new net DDRB_DQ2: U?.F2 (DQ2)
- new net DDRB_DQ3: U?.F8 (DQ3)
- new net DDRB_DQ4: U?.H3 (DQ4)
- new net DDRB_DQ5: U?.H8 (DQ5)
- new net DDRB_DQ6: U?.G2 (DQ6)
- new net DDRB_DQ7: U?.H7 (DQ7)
- new net DDRB_DQ8: U?.D7 (DQ8)
- new net DDRB_DQ9: U?.C3 (DQ9)
- new net DDRB_DQS0+: U?.F3 (LDQS)
- new net DDRB_DQS0-: U?.G3 (~{LDQS})
- new net DDRB_DQS1+: U?.C7 (UDQS)
- new net DDRB_DQS1-: U?.B7 (~{UDQS})
- new net DDR_ADDR0: U?.N3 (A0), U?.N3 (A0)
- new net DDR_ADDR1: U?.P7 (A1), U?.P7 (A1)
- new net DDR_ADDR10: U?.L7 (A10/AP), U?.L7 (A10/AP)
- new net DDR_ADDR11: U?.R7 (A11), U?.R7 (A11)
- new net DDR_ADDR12: U?.N7 (A12/~{BC}), U?.N7 (A12/~{BC})
- new net DDR_ADDR13: U?.T3 (A13), U?.T3 (A13)
- new net DDR_ADDR14: U?.T7 (A14), U?.T7 (A14)
- new net DDR_ADDR2: U?.P3 (A2), U?.P3 (A2)
- new net DDR_ADDR3: U?.N2 (A3), U?.N2 (A3)
- new net DDR_ADDR4: U?.P8 (A4), U?.P8 (A4)
- new net DDR_ADDR5: U?.P2 (A5), U?.P2 (A5)
- new net DDR_ADDR6: U?.R8 (A6), U?.R8 (A6)
- new net DDR_ADDR7: U?.R2 (A7), U?.R2 (A7)
- new net DDR_ADDR8: U?.T8 (A8), U?.T8 (A8)
- new net DDR_ADDR9: U?.R3 (A9), U?.R3 (A9)
- new net DDR_BA0: R?.2, U?.M2 (BA0), U?.M2 (BA0)
- new net DDR_BA1: R?.2, U?.N8 (BA1), U?.N8 (BA1)
- new net DDR_BA2: R?.2, U?.M3 (BA2), U?.M3 (BA2)
- new net DDR_CK+: U?.J7 (CK), U?.J7 (CK)
- new net DDR_CK-: U?.K7 (~{CK}), U?.K7 (~{CK})
- new net DDR_CKE: R?.2, U?.K9 (CKE), U?.K9 (CKE)
- new net DDR_ODT0: R?.2, U?.K1 (ODT), U?.K1 (ODT)
- new net DDR_nCAS: R?.2, U?.K3 (~{CAS}), U?.K3 (~{CAS})
- new net DDR_nCS: R?.2, U?.L2 (~{CS}), U?.L2 (~{CS})
- new net DDR_nRAS: R?.2, U?.J3 (~{RAS}), U?.J3 (~{RAS})
- new net DDR_nRST: U?.T2 (~{RESET}), U?.T2 (~{RESET})
- new net DDR_nWE: R?.2, U?.L3 (~{WE}), U?.L3 (~{WE})
- new net GND: C?.2, C?.2, C?.2, C?.2, R?.2, R?.2, U?.A9 (VSS), U?.A9 (VSS), U?.B1 (VSSQ), U?.B1 (VSSQ), U?.B3 (VSS), U?.B3 (VSS), U?.B9 (VSSQ), U?.B9 (VSSQ), U?.D1 (VSSQ), U?.D1 (VSSQ), U?.D8 (VSSQ), U?.D8 (VSSQ), U?.E1 (VSS), U?.E1 (VSS), U?.E2 (VSSQ), U?.E2 (VSSQ), U?.E8 (VSSQ), U?.E8 (VSSQ), U?.F9 (VSSQ), U?.F9 (VSSQ), U?.G1 (VSSQ), U?.G1 (VSSQ), U?.G8 (VSS), U?.G8 (VSS), U?.G9 (VSSQ), U?.G9 (VSSQ), U?.J2 (VSS), U?.J2 (VSS), U?.J8 (VSS), U?.J8 (VSS), U?.M1 (VSS), U?.M1 (VSS), U?.M9 (VSS), U?.M9 (VSS), U?.P1 (VSS), U?.P1 (VSS), U?.P9 (VSS), U?.P9 (VSS), U?.T1 (VSS), U?.T1 (VSS), U?.T9 (VSS), U?.T9 (VSS)

Commit message: ps progress; added ftdi; mezz pinout pedinging;
Parts:
- removed R? (x24): RT0402FRE0740R2L, Resistor_SMD:R_0402_1005Metric, symbol Resistors:RT0402FRE0740R2L
- added C? (x38): CL05B473KA5VPNC, Capacitor_SMD:C_0402_1005Metric, symbol Capacitors:CL05B473KA5VPNC
Connections:
- net +VCC_1V5: now also C?.1, C?.1, C?.1, C?.1, C?.1, C?.1, C?.1, C?.1, C?.1, C?.1, C?.1, C?.1, C?.1, C?.1, C?.1, C?.1, C?.1, C?.1, C?.1, C?.1, C?.1, C?.1, C?.1, C?.1, C?.1, C?.1, C?.1, C?.1, C?.1, C?.1, C?.1, C?.1, C?.1, C?.1, C?.1, C?.1, C?.1, C?.1
- net GND: now also C?.2, C?.2, C?.2, C?.2, C?.2, C?.2, C?.2, C?.2, C?.2, C?.2, C?.2, C?.2, C?.2, C?.2, C?.2, C?.2, C?.2, C?.2, C?.2, C?.2, C?.2, C?.2, C?.2, C?.2, C?.2, C?.2, C?.2, C?.2, C?.2, C?.2, C?.2, C?.2, C?.2, C?.2, C?.2, C?.2, C?.2, C?.2
Other:
- moved on the sheet: C?, R?, U?

Commit message: some ddr routing progress; layerstack per pcbway standard options, review reqd; commit prior to ddr split;
Parts:
- gave numbers to parts that had none: 46

Commit message: added starage, usb sch; more design progress in sch;
Parts:
- removed C121, C122, C123, C124, C125, C131, C132, C133, C134, C135, C141, C142, C143, C144, C145, C151, C152, C153, C154: CL05B473KA5VPNC, Capacitor_SMD:C_0402_1005Metric, symbol Capacitors:CL05B473KA5VPNC
- removed C159, C160: CL05B103KB5NNNC, Capacitor_SMD:C_0402_1005Metric, symbol Capacitors:CL05B103KB5NNNC
- removed R121: RC0402FR-07240RL, Resistor_SMD:R_0402_1005Metric, symbol Resistors:RC0402FR-07240RL
- removed U9: AS4C256M16D3C-12BCN, Package_BGA:BGA-96_9.0x13.0mm_Layout2x3x16_P0.8mm, symbol Memory_RAM:AS4C256M16D3
- renumbered C126 to C164, C127 to C165, C128 to C166, C129 to C167, C130 to C168, C136 to C169, C137 to C170, C138 to C171, C139 to C172, C140 to C173, C146 to C174, C147 to C175, C148 to C176, C149 to C177, C150 to C178, C155 to C179, C156 to C180, C157 to C181, C158 to C182, C161 to C183, C162 to C184, R122 to R123, U11 to U9
Connections:
- net DDRB_DM0 is gone; now on net DDRA_DM0: U9.E7 (LDM)
- net DDRB_DM1 is gone; now on net DDRA_DM1: U9.D3 (UDM)
- net DDRB_DQ0 is gone; now on net DDRA_DQ0: U9.E3 (DQ0)
- net DDRB_DQ1 is gone; now on net DDRA_DQ1: U9.F7 (DQ1)
- net DDRB_DQ10 is gone; now on net DDRA_DQ10: U9.C8 (DQ10)
- net DDRB_DQ11 is gone; now on net DDRA_DQ11: U9.C2 (DQ11)
- net DDRB_DQ12 is gone; now on net DDRA_DQ12: U9.A7 (DQ12)
- net DDRB_DQ13 is gone; now on net DDRA_DQ13: U9.A2 (DQ13)
- net DDRB_DQ14 is gone; now on net DDRA_DQ14: U9.B8 (DQ14)
- net DDRB_DQ15 is gone; now on net DDRA_DQ15: U9.A3 (DQ15)
- net DDRB_DQ2 is gone; now on net DDRA_DQ2: U9.F2 (DQ2)
- net DDRB_DQ3 is gone; now on net DDRA_DQ3: U9.F8 (DQ3)
- net DDRB_DQ4 is gone; now on net DDRA_DQ4: U9.H3 (DQ4)
- net DDRB_DQ5 is gone; now on net DDRA_DQ5: U9.H8 (DQ5)
- net DDRB_DQ6 is gone; now on net DDRA_DQ6: U9.G2 (DQ6)
- net DDRB_DQ7 is gone; now on net DDRA_DQ7: U9.H7 (DQ7)
- net DDRB_DQ8 is gone; now on net DDRA_DQ8: U9.D7 (DQ8)
- net DDRB_DQ9 is gone; now on net DDRA_DQ9: U9.C3 (DQ9)
- net DDRB_DQS0+ is gone; now on net DDRA_DQS0+: U9.F3 (LDQS)
- net DDRB_DQS0- is gone; now on net DDRA_DQS0-: U9.G3 (~{LDQS})
- net DDRB_DQS1+ is gone; now on net DDRA_DQS1+: U9.C7 (UDQS)
- net DDRB_DQS1- is gone; now on net DDRA_DQS1-: U9.B7 (~{UDQS})
Other:
- moved on the sheet: C164, C165, C166, C167, C168, C169, C170, C171, C172, C173, C174, C175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
