File: Hardware/Design Files/rfsom-01/mezzanine.kicad_sch (KiCad schematic)
At the start: 30 parts

Commit message: ddr progress; added more conns;
Parts:
- gave numbers to parts that had none: 30
Changed lines of the file:
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@@
 		(on_board yes)
 		(dnp no)
-		(property "Reference" "L?"
+		(property "Reference" "L5"
 			(at 237.49 80.01 0)
 			(effects
@@
 			(project "rfsom-01"
 				(path "/5dade83d-850c-4336-8f49-e0e8e6ebca37/aa769d64-0dd0-48a6-88b3-65c6d6ecbe65"
-					(reference "L?")
+					(reference "L5")
 					(unit 1)
 				)
@@
 		(on_board yes)
 		(dnp no)
-		(property "Reference" "L?"
+		(property "Reference" "L7"
 			(at 237.49 69.85 0)
 			(effects
@@
 			(project "rfsom-01"
 				(path "/5dade83d-850c-4336-8f49-e0e8e6ebca37/aa769d64-0dd0-48a6-88b3-65c6d6ecbe65"
-					(reference "L?")
+					(reference "L7")
 					(unit 1)
 				)
@@
 		(dnp yes)
 		(fields_autoplaced yes)
-		(property "Reference" "R?"
+		(property "Reference" "R13"
 			(at 91.44 67.3099 0)
 			(effects
@@
 			(project "rfsom-01"
 				(path "/5dade83d-850c-4336-8f49-e0e8e6ebca37/aa769d64-0dd0-48a6-88b3-65c6d6ecbe65"
-					(reference "R?")
+					(reference "R13")
 					(unit 1)
 				)
@@
 		(dnp no)
 		(fields_autoplaced yes)
-		(property "Reference" "R?"
+		(property "Reference" "R22"
 			(at 238.76 114.2999 0)
 			(effects
@@
 			(project "rfsom-01"
 				(path "/5dade83d-850c-4336-8f49-e0e8e6ebca37/aa769d64-0dd0-48a6-88b3-65c6d6ecbe65"
-					(reference "R?")
+					(reference "R22")
 					(unit 1)
 				)
@@
 		(dnp no)
 		(fields_autoplaced yes)
-		(property "Reference" "R?"
+		(property "Reference" "R7"
 			(at 30.48 80.0099 0)
 			(effects
@@
 			(project "rfsom-01"
 				(path "/5dade83d-850c-4336-8f49-e0e8e6ebca37/aa769d64-0dd0-48a6-88b3-65c6d6ecbe65"
-					(reference "R?")
+					(reference "R7")
 					(unit 1)
 				)
@@
 		(dnp yes)
 		(fields_autoplaced yes)
-		(property "Reference" "R?"
+		(property "Reference" "R15"
 			(at 91.44 110.4899 0)
 			(effects
@@
 			(project "rfsom-01"
 				(path "/5dade83d-850c-4336-8f49-e0e8e6ebca37/aa769d64-0dd0-48a6-88b3-65c6d6ecbe65"
-					(reference "R?")
+					(reference "R15")
 					(unit 1)
 				)
@@
 		(dnp no)
 		(fields_autoplaced yes)
-		(property "Reference" "C?"
+		(property "Reference" "C17"
 			(at 115.57 40.6399 0)
 			(effects
@@
 			(project "rfsom-01"
 				(path "/5dade83d-850c-4336-8f49-e0e8e6ebca37/aa769d64-0dd0-48a6-88b3-65c6d6ecbe65"
-					(reference "C?")
+					(reference "C17")
 					(unit 1)
 				)
@@
 		(dnp no)
 		(fields_autoplaced yes)
-		(property "Reference" "R?"
+		(property "Reference" "R14"
 			(at 91.44 80.0099 0)
 			(effects
@@
 			(project "rfsom-01"
 				(path "/5dade83d-850c-4336-8f49-e0e8e6ebca37/aa769d64-0dd0-48a6-88b3-65c6d6ecbe65"
-					(reference "R?")
+					(reference "R14")
 					(unit 1)
 				)
@@
 		(dnp no)
 		(fields_autoplaced yes)
-		(property "Reference" "R?"
+		(property "Reference" "R6"
 			(at 30.48 67.3099 0)
 			(effects
@@
 			(project "rfsom-01"
 				(path "/5dade83d-850c-4336-8f49-e0e8e6ebca37/aa769d64-0dd0-48a6-88b3-65c6d6ecbe65"
-					(reference "R?")
+					(reference "R6")
 					(unit 1)
 				)
@@
 		(on_board yes)
 		(dnp no)
-		(property "Reference" "L?"
+		(property "Reference" "L6"
 			(at 237.49 97.79 0)
 			(effects
@@
 			(project "rfsom-01"
 				(path "/5dade83d-850c-4336-8f49-e0e8e6ebca37/aa769d64-0dd0-48a6-88b3-65c6d6ecbe65"
-					(reference "L?")
+					(reference "L6")
 					(unit 1)
 				)
@@
 		(dnp yes)
 		(fields_autoplaced yes)
-		(property "Reference" "R?"
+		(property "Reference" "R12"
 			(at 62.23 123.1899 0)
 			(effects
@@
 			(project "rfsom-01"
 				(path "/5dade83d-850c-4336-8f49-e0e8e6ebca37/aa769d64-0dd0-48a6-88b3-65c6d6ecbe65"
-					(reference "R?")
+					(reference "R12")
 					(unit 1)
 				)
@@
 		(dnp no)
 		(fields_autoplaced yes)
-		(property "Reference" "C?"
+		(property "Reference" "C16"
 			(at 102.87 40.6399 0)
 			(effects
@@
 			(project "rfsom-01"
 				(path "/5dade83d-850c-4336-8f49-e0e8e6ebca37/aa769d64-0dd0-48a6-88b3-65c6d6ecbe65"
-					(reference "C?")
+					(reference "C16")
 					(unit 1)
 				)
@@
 		(dnp no)
 		(fields_autoplaced yes)
-		(property "Reference" "C?"
+		(property "Reference" "C20"
 			(at 140.97 40.6399 0)
 			(effects
@@
 			(project "rfsom-01"
 				(path "/5dade83d-850c-4336-8f49-e0e8e6ebca37/aa769d64-0dd0-48a6-88b3-65c6d6ecbe65"
-					(reference "C?")
+					(reference "C20")
 					(unit 1)
 				)
@@
 		(dnp yes)
 		(fields_autoplaced yes)
-		(property "Reference" "R?"
+		(property "Reference" "R18"
 			(at 91.44 166.3699 0)
 			(effects
@@
 			(project "rfsom-01"
 				(path "/5dade83d-850c-4336-8f49-e0e8e6ebca37/aa769d64-0dd0-48a6-88b3-65c6d6ecbe65"
-					(reference "R?")
+					(reference "R18")
 					(unit 1)
 				)
@@
 		(dnp no)
 		(fields_autoplaced yes)
-		(property "Reference" "R?"
+		(property "Reference" "R23"
 			(at 248.92 114.2999 0)
 			(effects
@@
 			(project "rfsom-01"
 				(path "/5dade83d-850c-4336-8f49-e0e8e6ebca37/aa769d64-0dd0-48a6-88b3-65c6d6ecbe65"
-					(reference "R?")
+					(reference "R23")
 					(unit 1)
 				)
@@
 		(on_board yes)
 		(dnp no)
-		(property "Reference" "R?"
+		(property "Reference" "R21"
 			(at 167.386 91.694 90)
 			(effects
@@
 			(project "rfsom-01"
 				(path "/5dade83d-850c-4336-8f49-e0e8e6ebca37/aa769d64-0dd0-48a6-88b3-65c6d6ecbe65"
-					(reference "R?")
+					(reference "R21")
 					(unit 1)
 				)
@@
 		(dnp no)
 		(fields_autoplaced yes)
-		(property "Reference" "C?"
+		(property "Reference" "C22"
 			(at 170.18 40.6399 0)
 			(effects
@@
 			(project "rfsom-01"
 				(path "/5dade83d-850c-4336-8f49-e0e8e6ebca37/aa769d64-0dd0-48a6-88b3-65c6d6ecbe65"
-					(reference "C?")
+					(reference "C22")
 					(unit 1)
 				)
@@
 		(dnp no)
 		(fields_autoplaced yes)
-		(property "Reference" "R?"
+		(property "Reference" "R16"
 			(at 91.44 123.1899 0)
 			(effects
@@
 			(project "rfsom-01"
 				(path "/5dade83d-850c-4336-8f49-e0e8e6ebca37/aa769d64-0dd0-48a6-88b3-65c6d6ecbe65"
-					(reference "R?")
+					(reference "R16")
 					(unit 1)
 				)
@@
 		(on_board yes)
 		(dnp no)
-		(property "Reference" "C?"
+		(property "Reference" "C23"
 			(at 171.45 78.486 90)
 			(effects
@@
 			(project "rfsom-01"
 				(path "/5dade83d-850c-4336-8f49-e0e8e6ebca37/aa769d64-0dd0-48a6-88b3-65c6d6ecbe65"
-					(reference "C?")
+					(reference "C23")
 					(unit 1)
 				)
@@
 		(dnp no)
 		(fields_autoplaced yes)
-		(property "Reference" "R?"
+		(property "Reference" "R11"
 			(at 62.23 110.4899 0)
 			(effects
@@
 			(project "rfsom-01"
 				(path "/5dade83d-850c-4336-8f49-e0e8e6ebca37/aa769d64-0dd0-48a6-88b3-65c6d6ecbe65"
-					(reference "R?")
+					(reference "R11")
 					(unit 1)
 				)
@@
 		(on_board yes)
 		(dnp no)
-		(property "Reference" "C?"
+		(property "Reference" "C19"
 			(at 127 92.202 0)
 			(effects
@@
 			(project "rfsom-01"
 				(path "/5dade83d-850c-4336-8f49-e0e8e6ebca37/aa769d64-0dd0-48a6-88b3-65c6d6ecbe65"
-					(reference "C?")
+					(reference "C19")
 					(unit 1)
 				)
@@
 		(on_board yes)
 		(dnp no)
-		(property "Reference" "C?"
+		(property "Reference" "C21"
 			(at 152.4 109.982 0)
 			(effects
@@
 			(project "rfsom-01"
 				(path "/5dade83d-850c-4336-8f49-e0e8e6ebca37/aa769d64-0dd0-48a6-88b3-65c6d6ecbe65"
-					(reference "C?")
+					(reference "C21")
 					(unit 1)
 				)
@@
 		(dnp no)
 		(fields_autoplaced yes)
-		(property "Reference" "R?"
+		(property "Reference" "R9"
 			(at 62.23 67.3099 0)
 			(effects
@@
 			(project "rfsom-01"
 				(path "/5dade83d-850c-4336-8f49-e0e8e6ebca37/aa769d64-0dd0-48a6-88b3-65c6d6ecbe65"
-					(reference "R?")
+					(reference "R9")
 					(unit 1)
 				)
@@
 		(dnp no)
 		(fields_autoplaced yes)
-		(property "Reference" "R?"
+		(property "Reference" "R17"
 			(at 91.44 153.6699 0)
 			(effects
@@
 			(project "rfsom-01"
 				(path "/5dade83d-850c-4336-8f49-e0e8e6ebca37/aa769d64-0dd0-48a6-88b3-65c6d6ecbe65"
-					(reference "R?")
+					(reference "R17")
 					(unit 1)
 				)
@@
 		(dnp no)
 		(fields_autoplaced yes)
-		(property "Reference" "R?"
+		(property "Reference" "R20"
 			(at 160.02 29.21 90)
 			(effects
@@
 			(project "rfsom-01"
 				(path "/5dade83d-850c-4336-8f49-e0e8e6ebca37/aa769d64-0dd0-48a6-88b3-65c6d6ecbe65"
-					(reference "R?")
+					(reference "R20")
 					(unit 1)
 				)
@@
 		(dnp no)
 		(fields_autoplaced yes)
-		(property "Reference" "U?"
+		(property "Reference" "U7"
 			(at 196.85 43.18 0)
 			(effects
@@
 			(project "rfsom-01"
 				(path "/5dade83d-850c-4336-8f49-e0e8e6ebca37/aa769d64-0dd0-48a6-88b3-65c6d6ecbe65"
-					(reference "U?")
+					(reference "U7")
 					(unit 1)
 				)
@@
 		(dnp no)
 		(fields_autoplaced yes)
-		(property "Reference" "R?"
+		(property "Reference" "R19"
 			(at 148.59 64.77 90)
 			(effects
@@
 			(project "rfsom-01"
 				(path "/5dade83d-850c-4336-8f49-e0e8e6ebca37/aa769d64-0dd0-48a6-88b3-65c6d6ecbe65"
-					(reference "R?")
+					(reference "R19")
 					(unit 1)
 				)
@@
 		(dnp no)
 		(fields_autoplaced yes)
-		(property "Reference" "R?"
+		(property "Reference" "R8"
 			(at 30.48 92.7099 0)
 			(effects
@@
 			(project "rfsom-01"
 				(path "/5dade83d-850c-4336-8f49-e0e8e6ebca37/aa769d64-0dd0-48a6-88b3-65c6d6ecbe65"
-					(reference "R?")
+					(reference "R8")
 					(unit 1)
 				)
@@
 		(dnp yes)
 		(fields_autoplaced yes)
-		(property "Reference" "R?"
+		(property "Reference" "R10"
 			(at 62.23 80.0099 0)
 			(effects
@@
 			(project "rfsom-01"
 				(path "/5dade83d-850c-4336-8f49-e0e8e6ebca37/aa769d64-0dd0-48a6-88b3-65c6d6ecbe65"
-					(reference "R?")
+					(reference "R10")
 					(unit 1)
 				)
@@
 		(dnp no)
 		(fields_autoplaced yes)
-		(property "Reference" "C?"
+		(property "Reference" "C18"
 			(at 128.27 40.6399 0)
 			(effects
@@
 			(project "rfsom-01"
 				(path "/5dade83d-850c-4336-8f49-e0e8e6ebca37/aa769d64-0dd0-48a6-88b3-65c6d6ecbe65"
-					(reference "C?")
+					(reference "C18")
 					(unit 1)
 				)

Commit message: ps progress; added ftdi; mezz pinout pedinging;
Parts:
- removed C16, C22: CL10B105KA8NNNC, Capacitor_SMD:C_0603_1608Metric_Pad1.08x0.95mm_HandSolder, symbol Capacitors:CL10B105KA8NNNC
- removed C17, C18, C20: CL31A106KBHNNNE, Capacitor_SMD:C_1206_3216Metric_Pad1.33x1.80mm_HandSolder, symbol Capacitors:CL31A106KBHNNNE
- removed C19, C21: CL05B104KA5NNNC, Capacitor_SMD:C_0402_1005Metric_Pad0.74x0.62mm_HandSolder, symbol Capacitors:CL05B104KA5NNNC
- removed C23: C0402C152J5GACTU, Capacitor_SMD:C_0402_1005Metric_Pad0.74x0.62mm_HandSolder, symbol Capacitors:C0402C152J5GACTU
- removed L5, L6, L7: 74404043022A, Inductors:WE-LQS, symbol Inductors:74404043022A
- removed R10, R11, R12, R13, R14, R15, R16, R17, R18, R9: RC0402FR-070RL, Resistor_SMD:R_0402_1005Metric_Pad0.72x0.64mm_HandSolder, symbol Resistors:RC0402FR-070RL
- removed R19, R22, R23: RC0402FR-07100KL, Resistor_SMD:R_0402_1005Metric_Pad0.72x0.64mm_HandSolder, symbol Resistors:RC0402FR-07100KL
- removed R20: RC0603FR-0710RL, Resistor_SMD:R_0603_1608Metric_Pad0.98x0.95mm_HandSolder, symbol Resistors:RC0603FR-0710RL
- removed R21, R7: RC0603FR-07100KL, Resistor_SMD:R_0603_1608Metric_Pad0.98x0.95mm_HandSolder, symbol Resistors:RC0603FR-07100KL
- removed R6: RC0603FR-071M2L, Resistor_SMD:R_0603_1608Metric_Pad0.98x0.95mm_HandSolder, symbol Resistors:RC0603FR-071M2L
- removed R8: RC0603FR-07499KL, Resistor_SMD:R_0603_1608Metric_Pad0.98x0.95mm_HandSolder, symbol Resistors:RC0603FR-07499KL
- removed U7: TPS65023BRSBR, ICs:RSB0040B, symbol ICs:TPS65023BRSBR
- added J? (x2): DF40C-80DP-0.4V(58), Connectors:DF40C-80DP-0.4V, symbol Connectors:DF40C-80DP-0.4V(58)
- added J?: DF40C-70DP-0.4V(51), symbol Connectors:DF40C-70DP-0.4V(51)
Connections:
- net GND: now also J?.11, J?.14, J?.17, J?.2, J?.20, J?.23, J?.26, J?.35, J?.36, J?.5, J?.72, J?.74, J?.76, J?.78, J?.8, J?.80
- new net +VIN_5V0: J?.71, J?.73, J?.75, J?.77, J?.79
Other:
- note removed: "1.2A"
- note removed: "1.2V"
- note removed: "1.5A"
- note removed: "1.6V"
- note removed: "1.8V"
- note removed: "1A"
- note removed: "1V 1.35V 3.3V 1.8V LDO 1.8V"
- note removed: "200mA"
- note removed: "3.3V"
- note removed: "DEFLDO1 DEFLDO2 VLDO1 VLDO2 0 0 1.3 V 3.3 V 0 1 1.3 V 1.8 V 1 0 2.8 V 3.3 V 1 1 1.8 V 3.3 V"
- note removed: "PLACE JUMPERS OVERLAPPED."

Commit message: some ddr routing progress; layerstack per pcbway standard options, review reqd; commit prior to ddr split;
Parts:
- J4: renamed from J?; footprint (none) -> Connectors:DF40C-70DP-0.4V
- gave numbers to parts that had none: 2
Connections:
- net EXT_ETH_TRX3-: now reaches J5.1
- net EXT_ETH_TRX1-: now reaches J5.13
- net EXT_ETH_TRX1+: now reaches J5.15
- net EXT_ETH_TRX0-: now reaches J5.19
- net EXT_ETH_TRX0+: now reaches J5.21
- net EXT_ETH_LED-LINK: now reaches J5.25
- net EXT_ETH_LED-ACT: now reaches J5.27
- net EXT_ETH_TRX3+: now reaches J5.3
- net EXT_ETH_TRX2-: now reaches J5.7
- net EXT_ETH_TRX2+: now reaches J5.9
Changed lines of the file:
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@@
+	(wire
+		(pts
+			(xy 243.84 67.31) (xy 232.41 67.31)
+		)
+		(stroke
+			(width 0)
+			(type default)
+		)
+	)
 	(wire
 		(pts
@@
 	(wire
 		(pts
+			(xy 243.84 44.45) (xy 232.41 44.45)
+		)
+		(stroke
+			(width 0)
+			(type default)
+		)
+	)
+	(wire
+		(pts
 			(xy 247.65 130.81) (xy 247.65 133.35)
 		)
@@
 	(wire
 		(pts
+			(xy 243.84 41.91) (xy 232.41 41.91)
+		)
+		(stroke
+			(width 0)
+			(type default)
+		)
+	)
+	(wire
+		(pts
 			(xy 215.9 72.39) (xy 222.25 72.39)
 		)
@@
 	(wire
 		(pts
+			(xy 243.84 72.39) (xy 232.41 72.39)
+		)
+		(stroke
+			(width 0)
+			(type default)
+		)
+	)
+	(wire
+		(pts
 			(xy 215.9 138.43) (xy 215.9 140.97)
 		)
@@
 	(wire
 		(pts
+			(xy 243.84 52.07) (xy 232.41 52.07)
+		)
+		(stroke
+			(width 0)
+			(type default)
+		)
+	)
+	(wire
+		(pts
 			(xy 215.9 72.39) (xy 215.9 85.09)
 		)
@@
 	(wire
 		(pts
+			(xy 243.84 64.77) (xy 232.41 64.77)
+		)
+		(stroke
+			(width 0)
+			(type default)
+		)
+	)
+	(wire
+		(pts
 			(xy 215.9 140.97) (xy 222.25 140.97)
 		)
@@
 	(wire
 		(pts
+			(xy 243.84 74.93) (xy 232.41 74.93)
+		)
+		(stroke
+			(width 0)
+			(type default)
+		)
+	)
+	(wire
+		(pts
 			(xy 215.9 85.09) (xy 215.9 130.81)
 		)
@@
 	(wire
 		(pts
+			(xy 243.84 57.15) (xy 232.41 57.15)
+		)
+		(stroke
+			(width 0)
+			(type default)
+		)
+	)
+	(wire
+		(pts
 			(xy 232.41 46.99) (xy 238.76 46.99)
 		)
@@
 			(width 0)
 			(type default)
+		)
+	)
+	(wire
+		(pts
+			(xy 243.84 49.53) (xy 232.41 49.53)
+		)
+		(stroke
+			(width 0)
+			(type default)
+		)
+	)
+	(wire
+		(pts
+			(xy 243.84 59.69) (xy 232.41 59.69)
+		)
+		(stroke
+			(width 0)
+			(type default)
+		)
+	)
+	(hierarchical_label "EXT_ETH_TRX3+"
+		(shape bidirectional)
+		(at 243.84 44.45 0)
+		(effects
+			(font
+				(size 1.27 1.27)
+			)
+			(justify left)
+		)
+	)
+	(hierarchical_label "EXT_ETH_LED-LINK"
+		(shape input)
+		(at 243.84 72.39 0)
+		(effects
+			(font
+				(size 1.27 1.27)
+			)
+			(justify left)
+		)
+	)
+	(hierarchical_label "EXT_ETH_TRX1+"
+		(shape bidirectional)
+		(at 243.84 59.69 0)
+		(effects
+			(font
+				(size 1.27 1.27)
+			)
+			(justify left)
+		)
+	)
+	(hierarchical_label "EXT_ETH_TRX3-"
+		(shape bidirectional)
+		(at 243.84 41.91 0)
+		(effects
+			(font
+				(size 1.27 1.27)
+			)
+			(justify left)
+		)
+	)
+	(hierarchical_label "EXT_ETH_TRX2+"
+		(shape bidirectional)
+		(at 243.84 52.07 0)
+		(effects
+			(font
+				(size 1.27 1.27)
+			)
+			(justify left)
+		)
+	)
+	(hierarchical_label "EXT_ETH_TRX0-"
+		(shape bidirectional)
+		(at 243.84 64.77 0)
+		(effects
+			(font
+				(size 1.27 1.27)
+			)
+			(justify left)
+		)
+	)
+	(hierarchical_label "EXT_ETH_TRX0+"
+		(shape bidirectional)
+		(at 243.84 67.31 0)
+		(effects
+			(font
+				(size 1.27 1.27)
+			)
+			(justify left)
+		)
+	)
+	(hierarchical_label "EXT_ETH_TRX1-"
+		(shape bidirectional)
+		(at 243.84 57.15 0)
+		(effects
+			(font
+				(size 1.27 1.27)
+			)
+			(justify left)
+		)
+	)
+	(hierarchical_label "EXT_ETH_TRX2-"
+		(shape bidirectional)
+		(at 243.84 49.53 0)
+		(effects
+			(font
+				(size 1.27 1.27)
+			)
+			(justify left)
+		)
+	)
+	(hierarchical_label "EXT_ETH_LED-ACT"
+		(shape input)
+		(at 243.84 74.93 0)
+		(effects
+			(font
+				(size 1.27 1.27)
+			)
+			(justify left)
 		)
 	)
@@
 		(on_board yes)
 		(dnp no)
-		(property "Reference" "J?"
+		(property "Reference" "J5"
 			(at 227.33 34.29 0)
 			(effects
@@
 			(project "rfsom-01"
 				(path "/5dade83d-850c-4336-8f49-e0e8e6ebca37/aa769d64-0dd0-48a6-88b3-65c6d6ecbe65"
-					(reference "J?")
+					(reference "J5")
 					(unit 1)
 				)
@@
 		(on_board yes)
 		(dnp no)
-		(property "Reference" "J?"
+		(property "Reference" "J4"
 			(at 132.08 45.72 0)
 			(effects
@@
 			)
 		)
-		(property "Footprint" ""
+		(property "Footprint" "Connectors:DF40C-70DP-0.4V"
 			(at 134.62 50.8 0)
 			(effects
@@
 			(project ""
 				(path "/5dade83d-850c-4336-8f49-e0e8e6ebca37/aa769d64-0dd0-48a6-88b3-65c6d6ecbe65"
-					(reference "J?")
+					(reference "J4")
 					(unit 1)
 				)
@@
 		(on_board yes)
 		(dnp no)
-		(property "Reference" "J?"
+		(property "Reference" "J3"
 			(at 48.26 39.37 0)
 			(effects
@@
 			(project ""
 				(path "/5dade83d-850c-4336-8f49-e0e8e6ebca37/aa769d64-0dd0-48a6-88b3-65c6d6ecbe65"
-					(reference "J?")
+					(reference "J3")
 					(unit 1)
 				)

Commit message: added starage, usb sch; more design progress in sch;
Parts:
- removed J3, J5: DF40C-80DP-0.4V(58), Connectors:DF40C-80DP-0.4V, symbol Connectors:DF40C-80DP-0.4V(58)
- removed J4: DF40C-70DP-0.4V(51), Connectors:DF40C-70DP-0.4V, symbol Connectors:DF40C-70DP-0.4V(51)
- added J3, J4: Conn_01x06, symbol Connector_Generic:Conn_01x06
- added R135, R136: R, symbol Device:R
- added U15: FT232HQ-REEL, Package_DFN_QFN:QFN-48-1EP_7x7mm_P0.5mm_EP5.1x5.1mm, symbol Interface_USB:FT232H
Connections:
- net GND: now also J3.4 (Pin_4), J4.4 (Pin_4)
- new net AD0: J3.5 (Pin_5), U15.13 (ADBUS0)
- new net AD1: R135.1, U15.14 (ADBUS1)
- new net AD2: J3.3 (Pin_3), R135.2, U15.15 (ADBUS2)
- new net AD4: J3.2 (Pin_2), U15.17 (ADBUS4)
- new net BD0: J4.5 (Pin_5), U15.21 (ACBUS0)
- new net BD1: R136.1, U15.25 (ACBUS1)
- new net BD2: J4.3 (Pin_3), R136.2, U15.26 (ACBUS2)
- new net BD4: J4.2 (Pin_2), U15.28 (ACBUS4)
