File: Hardware/Design Files/rfsom-01/ram-pl.kicad_sch (KiCad schematic)
At the start: 35 parts, among them U12 TPS51200DRCR, U8 AS4C256M16D3C-12BCN

Commit message: updated sch pdf; routign progress;
Parts:
- C121, C122, C123, C124, C125, C131, C132, C133, C134, C135, C141, C142, C143, C144, C145, C151, C152, C153, C154, C159, C160, R121, U8: now not fitted
Connections:
- net DDRA_DM0 renamed DDR_DM0
- net DDRA_DM1 renamed DDR_DM1
- net DDRA_DQ0 renamed DDR_DQ0
- net DDRA_DQ1 renamed DDR_DQ1
- net DDRA_DQ10 renamed DDR_DQ10
- net DDRA_DQ11 renamed DDR_DQ11
- net DDRA_DQ12 renamed DDR_DQ12
- net DDRA_DQ13 renamed DDR_DQ13
- net DDRA_DQ14 renamed DDR_DQ14
- net DDRA_DQ15 renamed DDR_DQ15
- net DDRA_DQ2 renamed DDR_DQ2
- net DDRA_DQ3 renamed DDR_DQ3
- net DDRA_DQ4 renamed DDR_DQ4
- net DDRA_DQ5 renamed DDR_DQ5
- net DDRA_DQ6 renamed DDR_DQ6
- net DDRA_DQ7 renamed DDR_DQ7
- net DDRA_DQ8 renamed DDR_DQ8
- net DDRA_DQ9 renamed DDR_DQ9
- net DDRA_DQS0+ renamed DDR_DQS0+
- net DDRA_DQS0- renamed DDR_DQS0-
- net DDRA_DQS1+ renamed DDR_DQS1+
- net DDRA_DQS1- renamed DDR_DQS1-
Changed lines of the file:
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@@
 		)
 	)
-	(label "DDRA_DQ2"
+	(label "DDR_DQ2"
 		(at 105.41 41.91 180)
 		(effects
@@
 		)
 	)
-	(label "DDRA_DQ15"
+	(label "DDR_DQ15"
 		(at 105.41 74.93 180)
 		(effects
@@
 		)
 	)
-	(label "DDRA_DQ8"
+	(label "DDR_DQ8"
 		(at 105.41 57.15 180)
 		(effects
@@
 		)
 	)
-	(label "DDRA_DQ5"
+	(label "DDR_DQ5"
 		(at 105.41 49.53 180)
 		(effects
@@
 		)
 	)
-	(label "DDRA_DM1"
+	(label "DDR_DM1"
 		(at 105.41 82.55 180)
 		(effects
@@
 		)
 	)
-	(label "DDRA_DQ0"
+	(label "DDR_DQ0"
 		(at 105.41 36.83 180)
 		(effects
@@
 		)
 	)
-	(label "DDRA_DQ10"
+	(label "DDR_DQ10"
 		(at 105.41 62.23 180)
 		(effects
@@
 		)
 	)
-	(label "DDRA_DQ13"
+	(label "DDR_DQ13"
 		(at 105.41 69.85 180)
 		(effects
@@
 		)
 	)
-	(label "DDRA_DQ1"
+	(label "DDR_DQ1"
 		(at 105.41 39.37 180)
 		(effects
@@
 		)
 	)
-	(label "DDRA_DQ12"
+	(label "DDR_DQ12"
 		(at 105.41 67.31 180)
 		(effects
@@
 		)
 	)
-	(label "DDRA_DQ11"
+	(label "DDR_DQ11"
 		(at 105.41 64.77 180)
 		(effects
@@
 		)
 	)
-	(label "DDRA_DM0"
+	(label "DDR_DM0"
 		(at 105.41 80.01 180)
 		(effects
@@
 		)
 	)
-	(label "DDRA_DQ6"
+	(label "DDR_DQ6"
 		(at 105.41 52.07 180)
 		(effects
@@
 		)
 	)
-	(label "DDRA_DQ7"
+	(label "DDR_DQ7"
 		(at 105.41 54.61 180)
 		(effects
@@
 		)
 	)
-	(label "DDRA_DQ4"
+	(label "DDR_DQ4"
 		(at 105.41 46.99 180)
 		(effects
@@
 		)
 	)
-	(label "DDRA_DQ14"
+	(label "DDR_DQ14"
 		(at 105.41 72.39 180)
 		(effects
@@
 		)
 	)
-	(label "DDRA_DQ9"
+	(label "DDR_DQ9"
 		(at 105.41 59.69 180)
 		(effects
@@
 		)
 	)
-	(label "DDRA_DQ3"
+	(label "DDR_DQ3"
 		(at 105.41 44.45 180)
 		(effects
@@
 		)
 	)
-	(hierarchical_label "DDRA_DQ[0..15]"
+	(hierarchical_label "DDR_DQ[0..15]"
 		(shape bidirectional)
 		(at 111.76 30.48 0)
@@
 		)
 	)
-	(hierarchical_label "DDRA_DQS0+"
+	(hierarchical_label "DDR_DQS0+"
 		(shape input)
 		(at 105.41 87.63 0)
@@
 		)
 	)
-	(hierarchical_label "DDRA_DQS0-"
+	(hierarchical_label "DDR_DQS0-"
 		(shape input)
 		(at 105.41 90.17 0)
@@
 		)
 	)
-	(hierarchical_label "DDRA_DQS1-"
+	(hierarchical_label "DDR_DQS1-"
 		(shape input)
 		(at 105.41 95.25 0)
@@
 		)
 	)
-	(hierarchical_label "DDRA_DQS1+"
+	(hierarchical_label "DDR_DQS1+"
 		(shape input)
 		(at 105.41 92.71 0)
@@
 		)
 	)
-	(hierarchical_label "DDRA_DM[0..1]"
+	(hierarchical_label "DDR_DM[0..1]"
 		(shape bidirectional)
 		(at 113.03 74.93 0)
@@
 		(in_bom yes)
 		(on_board yes)
-		(dnp no)
+		(dnp yes)
 		(fields_autoplaced yes)
 		(property "Reference" "C160"
@@
 		(in_bom yes)
 		(on_board yes)
-		(dnp no)
+		(dnp yes)
 		(fields_autoplaced yes)
 		(property "Reference" "C121"
@@
 		(in_bom yes)
 		(on_board yes)
-		(dnp no)
+		(dnp yes)
 		(fields_autoplaced yes)
 		(property "Reference" "C153"
@@
 		(in_bom yes)
 		(on_board yes)
-		(dnp no)
+		(dnp yes)
 		(fields_autoplaced yes)
 		(property "Reference" "C134"
@@
 		(in_bom yes)
 		(on_board yes)
-		(dnp no)
+		(dnp yes)
 		(fields_autoplaced yes)
 		(property "Reference" "C143"
@@
 		(in_bom yes)
 		(on_board yes)
-		(dnp no)
+		(dnp yes)
 		(fields_autoplaced yes)
 		(property "Reference" "C152"
@@
 		(in_bom yes)
 		(on_board yes)
-		(dnp no)
+		(dnp yes)
 		(fields_autoplaced yes)
 		(property "Reference" "C154"
@@
 		(in_bom yes)
 		(on_board yes)
-		(dnp no)
+		(dnp yes)
 		(fields_autoplaced yes)
 		(property "Reference" "C123"
@@
 		(in_bom yes)
 		(on_board yes)
-		(dnp no)
+		(dnp yes)
 		(fields_autoplaced yes)
 		(property "Reference" "C132"
@@
 		(in_bom yes)
 		(on_board yes)
-		(dnp no)
+		(dnp yes)
 		(fields_autoplaced yes)
 		(property "Reference" "U8"
@@
 		(in_bom yes)
 		(on_board yes)
-		(dnp no)
+		(dnp yes)
 		(fields_autoplaced yes)
 		(property "Reference" "C124"
@@
 		(in_bom yes)
 		(on_board yes)
-		(dnp no)
+		(dnp yes)
 		(fields_autoplaced yes)
 		(property "Reference" "C159"
@@
 		(in_bom yes)
 		(on_board yes)
-		(dnp no)
+		(dnp yes)
 		(fields_autoplaced yes)
 		(property "Reference" "C144"
@@
 		(in_bom yes)
 		(on_board yes)
-		(dnp no)
+		(dnp yes)
 		(fields_autoplaced yes)
 		(property "Reference" "C122"
@@
 		(in_bom yes)
 		(on_board yes)
-		(dnp no)
+		(dnp yes)
 		(fields_autoplaced yes)
 		(property "Reference" "C125"
@@
 		(in_bom yes)
 		(on_board yes)
-		(dnp no)
+		(dnp yes)
 		(fields_autoplaced yes)
 		(property "Reference" "C133"
@@
 		(in_bom yes)
 		(on_board yes)
-		(dnp no)
+		(dnp yes)
 		(fields_autoplaced yes)
 		(property "Reference" "C131"
@@
 		(in_bom yes)
 		(on_board yes)
-		(dnp no)
+		(dnp yes)
 		(fields_autoplaced yes)
 		(property "Reference" "R121"
@@
 		(in_bom yes)
 		(on_board yes)
-		(dnp no)
+		(dnp yes)
 		(fields_autoplaced yes)
 		(property "Reference" "C151"
@@
 		(in_bom yes)
 		(on_board yes)
-		(dnp no)
+		(dnp yes)
 		(fields_autoplaced yes)
 		(property "Reference" "C135"
@@
 		(in_bom yes)
 		(on_board yes)
-		(dnp no)
+		(dnp yes)
 		(fields_autoplaced yes)
 		(property "Reference" "C142"
@@
 		(in_bom yes)
 		(on_board yes)
-		(dnp no)
+		(dnp yes)
 		(fields_autoplaced yes)
 		(property "Reference" "C141"
@@
 		(in_bom yes)
 		(on_board yes)
-		(dnp no)
+		(dnp yes)
 		(fields_autoplaced yes)
 		(property "Reference" "C145"
