File: Hardware/Design Files/rfsom-01/rfsom-01.kicad_pcb (KiCad board)
At the start: 2 copper layers, 80 x 68.9 mm, 0 parts

Commit message: some ddr routing progress; layerstack per pcbway standard options, review reqd; commit prior to ddr split;
Parts:
- added C1: CL21B475KAFNNNE, Capacitor_SMD:C_0805_2012Metric, F.Cu at (83.1, 111.5)
- added C10: CL21B106KQQNFNE, Capacitor_SMD:C_0805_2012Metric, F.Cu at (108.8, 58.8)
- added C100: GRM188R70J474KA01D, Capacitor_SMD:C_0603_1608Metric, F.Cu at (156.4, 22.0)
- added C101: GRM188R70J474KA01D, Capacitor_SMD:C_0603_1608Metric, F.Cu at (156.4, 24.6)
- added C102: GRM188R70J474KA01D, Capacitor_SMD:C_0603_1608Metric, F.Cu at (156.4, 27.1)
- added C103: GRM188R70J474KA01D, Capacitor_SMD:C_0603_1608Metric, F.Cu at (156.4, 29.6)
- added C104: CL10B105KA8NNNC, Capacitor_SMD:C_0603_1608Metric, F.Cu at (193.3, 52.6)
- added C105: CL05B104KA5NNNC, Capacitor_SMD:C_0402_1005Metric, F.Cu at (205.9, 77.1)
- added C106: GRM188R70J474KA01D, Capacitor_SMD:C_0603_1608Metric, F.Cu at (193.3, 55.1)
- added C107: CL05B104KA5NNNC, Capacitor_SMD:C_0402_1005Metric, F.Cu at (205.9, 79.1)
- added C108: CL05B104KA5NNNC, Capacitor_SMD:C_0402_1005Metric, F.Cu at (205.9, 81.0)
- added C109: CL05B104KA5NNNC, Capacitor_SMD:C_0402_1005Metric, F.Cu at (205.9, 83.0)
- added C11: CL21B106KQQNFNE, Capacitor_SMD:C_0805_2012Metric, F.Cu at (110.8, 58.8)
- added C110: CL05B104KA5NNNC, Capacitor_SMD:C_0402_1005Metric, F.Cu at (205.9, 85.0)
- added C111: CL21B106KQQNFNE, Capacitor_SMD:C_0805_2012Metric, F.Cu at (234.7, 132.1)
- added C112: CL05B104KA5NNNC, Capacitor_SMD:C_0402_1005Metric, F.Cu at (225.3, 131.6)
- added C113: CL05B104KA5NNNC, Capacitor_SMD:C_0402_1005Metric, F.Cu at (225.3, 133.5)
- added C114: CL05B104KA5NNNC, Capacitor_SMD:C_0402_1005Metric, F.Cu at (225.3, 135.5)
- added C115: CL05B104KA5NNNC, Capacitor_SMD:C_0402_1005Metric, F.Cu at (228.2, 131.6)
- added C116: CL05B104KA5NNNC, Capacitor_SMD:C_0402_1005Metric, F.Cu at (228.2, 133.5)
- added C117: CL05B104KA5NNNC, Capacitor_SMD:C_0402_1005Metric, F.Cu at (228.2, 135.5)
- added C118: CL05B104KA5NNNC, Capacitor_SMD:C_0402_1005Metric, F.Cu at (231.0, 131.6)
- added C119: CL05B104KA5NNNC, Capacitor_SMD:C_0402_1005Metric, F.Cu at (231.0, 133.5)
- added C12: CL31A106KBHNNNE, Capacitor_SMD:C_1206_3216Metric, F.Cu at (76.9, 126.2)
- added C120: CL05B104KA5NNNC, Capacitor_SMD:C_0402_1005Metric, F.Cu at (231.0, 135.5)
- added C121: CL05B473KA5VPNC, Capacitor_SMD:C_0402_1005Metric, B.Cu at (104.8, 79.2)
- added C122: CL05B473KA5VPNC, Capacitor_SMD:C_0402_1005Metric, B.Cu at (110.1, 78.1)
- added C123: CL05B473KA5VPNC, Capacitor_SMD:C_0402_1005Metric, B.Cu at (113.8, 79.2)
- added C124: CL05B473KA5VPNC, Capacitor_SMD:C_0402_1005Metric, B.Cu at (103.9, 71.8)
- added C125: CL05B473KA5VPNC, Capacitor_SMD:C_0402_1005Metric, B.Cu at (105.8, 70.8)
- added C126: CL05B473KA5VPNC, Capacitor_SMD:C_0402_1005Metric, B.Cu at (105.0, 90.3)
- added C127: CL05B473KA5VPNC, Capacitor_SMD:C_0402_1005Metric, B.Cu at (104.8, 88.5)
- added C128: CL05B473KA5VPNC, Capacitor_SMD:C_0402_1005Metric, B.Cu at (109.0, 84.0)
- added C129: CL05B473KA5VPNC, Capacitor_SMD:C_0402_1005Metric, B.Cu at (105.5, 81.8)
- added C13: CL31A106KBHNNNE, Capacitor_SMD:C_1206_3216Metric, F.Cu at (76.9, 136.8)
- added C130: CL05B473KA5VPNC, Capacitor_SMD:C_0402_1005Metric, B.Cu at (111.0, 86.1)
- added C131: CL05B473KA5VPNC, Capacitor_SMD:C_0402_1005Metric, B.Cu at (109.8, 70.8)
- added C132: CL05B473KA5VPNC, Capacitor_SMD:C_0402_1005Metric, B.Cu at (107.2, 72.2)
- added C133: CL05B473KA5VPNC, Capacitor_SMD:C_0402_1005Metric, B.Cu at (108.0, 70.8)
- added C134: CL05B473KA5VPNC, Capacitor_SMD:C_0402_1005Metric, B.Cu at (107.4, 77.2)
- added C135: CL05B473KA5VPNC, Capacitor_SMD:C_0402_1005Metric, B.Cu at (106.7, 79.2)
- added C136: CL05B473KA5VPNC, Capacitor_SMD:C_0402_1005Metric, B.Cu at (103.9, 82.8)
- added C137: CL05B473KA5VPNC, Capacitor_SMD:C_0402_1005Metric, B.Cu at (107.2, 83.2)
- added C138: CL05B473KA5VPNC, Capacitor_SMD:C_0402_1005Metric, B.Cu at (116.2, 90.3)
- added C139: CL05B473KA5VPNC, Capacitor_SMD:C_0402_1005Metric, B.Cu at (113.8, 90.3)
- added C14: CL31A106KBHNNNE, Capacitor_SMD:C_1206_3216Metric, F.Cu at (77.0, 136.8)
- added C14: CL31A106KBHNNNE, Capacitor_SMD:C_1206_3216Metric, F.Cu at (81.5, 126.2)
- added C140: CL05B473KA5VPNC, Capacitor_SMD:C_0402_1005Metric, B.Cu at (110.1, 89.2)
- added C141: CL05B473KA5VPNC, Capacitor_SMD:C_0402_1005Metric, B.Cu at (111.0, 75.0)
- added C142: CL05B473KA5VPNC, Capacitor_SMD:C_0402_1005Metric, B.Cu at (108.5, 79.2)
- added C143: CL05B473KA5VPNC, Capacitor_SMD:C_0402_1005Metric, B.Cu at (111.5, 78.5)
- added C144: CL05B473KA5VPNC, Capacitor_SMD:C_0402_1005Metric, B.Cu at (115.7, 79.2)
- added C145: CL05B473KA5VPNC, Capacitor_SMD:C_0402_1005Metric, B.Cu at (114.5, 70.8)
- added C146: CL05B473KA5VPNC, Capacitor_SMD:C_0402_1005Metric, B.Cu at (111.5, 89.5)
- added C147: CL05B473KA5VPNC, Capacitor_SMD:C_0402_1005Metric, B.Cu at (107.4, 88.2)
- added C148: CL05B473KA5VPNC, Capacitor_SMD:C_0402_1005Metric, B.Cu at (106.8, 90.3)
- added C149: CL05B473KA5VPNC, Capacitor_SMD:C_0402_1005Metric, B.Cu at (108.2, 81.8)
- added C15: CL31A106KBHNNNE, Capacitor_SMD:C_1206_3216Metric, F.Cu at (81.5, 136.8)
- added C150: CL05B473KA5VPNC, Capacitor_SMD:C_0402_1005Metric, B.Cu at (110.2, 81.8)
- added C151: CL05B473KA5VPNC, Capacitor_SMD:C_0402_1005Metric, B.Cu at (112.2, 72.8)
- added C152: CL05B473KA5VPNC, Capacitor_SMD:C_0402_1005Metric, B.Cu at (117.0, 70.8)
- added C153: CL05B473KA5VPNC, Capacitor_SMD:C_0402_1005Metric, B.Cu at (109.1, 72.8)
- added C154: CL05B473KA5VPNC, Capacitor_SMD:C_0402_1005Metric, B.Cu at (104.8, 77.3)
- added C155: CL05B473KA5VPNC, Capacitor_SMD:C_0402_1005Metric, B.Cu at (108.7, 90.3)
- added C156: CL05B473KA5VPNC, Capacitor_SMD:C_0402_1005Metric, B.Cu at (116.3, 81.8)
- added C157: CL05B473KA5VPNC, Capacitor_SMD:C_0402_1005Metric, B.Cu at (114.5, 81.8)
- added C158: CL05B473KA5VPNC, Capacitor_SMD:C_0402_1005Metric, B.Cu at (112.2, 84.0)
- added C159: CL05B103KB5NNNC, Capacitor_SMD:C_0402_1005Metric, F.Cu at (188.4, 110.9)
- added C16: CL05B104KA5NNNC, Capacitor_SMD:C_0402_1005Metric, F.Cu at (212.2, 104.9)
- added C160: CL05B103KB5NNNC, Capacitor_SMD:C_0402_1005Metric, F.Cu at (188.4, 112.9)
- added C161: CL05B103KB5NNNC, Capacitor_SMD:C_0402_1005Metric, F.Cu at (188.4, 114.9)
- added C162: CL05B103KB5NNNC, Capacitor_SMD:C_0402_1005Metric, F.Cu at (188.4, 116.8)
- added C163: GRM188R70J474KA01D, Capacitor_SMD:C_0603_1608Metric, B.Cu at (133.9, 84.9)
- added C17: CL05B104KA5NNNC, Capacitor_SMD:C_0402_1005Metric, F.Cu at (212.2, 106.8)
- added C18: CL10B105KA8NNNC, Capacitor_SMD:C_0603_1608Metric, F.Cu at (200.7, 89.2)
- added C19: CL31A106KBHNNNE, Capacitor_SMD:C_1206_3216Metric, F.Cu at (216.5, 89.6)
- added C2: GRM188R60G106ME47, Capacitor_SMD:C_0603_1608Metric, F.Cu at (83.4, 107.2)
- added C20: CL05B104KA5NNNC, Capacitor_SMD:C_0402_1005Metric, F.Cu at (212.2, 108.8)
- added C21: CL05B104KA5NNNC, Capacitor_SMD:C_0402_1005Metric, F.Cu at (212.2, 110.8)
- added C22: CL05B104KA5NNNC, Capacitor_SMD:C_0402_1005Metric, F.Cu at (215.1, 102.9)
- added C23: CL05B104KA5NNNC, Capacitor_SMD:C_0402_1005Metric, F.Cu at (215.1, 104.9)
- added C24: CL05B104KA5NNNC, Capacitor_SMD:C_0402_1005Metric, F.Cu at (215.1, 106.8)
- added C25: CL21B475KAFNNNE, Capacitor_SMD:C_0805_2012Metric, F.Cu at (215.9, 99.5)
- added C26: CL31A106KBHNNNE, Capacitor_SMD:C_1206_3216Metric, F.Cu at (216.5, 93.0)
- added C27: CL05B104KA5NNNC, Capacitor_SMD:C_0402_1005Metric, F.Cu at (215.1, 108.8)
- added C28: CL05B103KB5NNNC, Capacitor_SMD:C_0402_1005Metric, F.Cu at (215.1, 110.8)
- added C29: CL31A106KBHNNNE, Capacitor_SMD:C_1206_3216Metric, F.Cu at (216.5, 96.3)
- added C3: CL21B475KPFNNNE, Capacitor_SMD:C_0805_2012Metric, F.Cu at (103.8, 48.9)
- added C30: CL05B104KA5NNNC, Capacitor_SMD:C_0402_1005Metric, F.Cu at (217.9, 102.9)
- added C31: CL05B104KA5NNNC, Capacitor_SMD:C_0402_1005Metric, F.Cu at (217.9, 104.9)
- added C32: CL05B104KA5NNNC, Capacitor_SMD:C_0402_1005Metric, F.Cu at (217.9, 106.8)
- added C33: CL21B475KAFNNNE, Capacitor_SMD:C_0805_2012Metric, F.Cu at (264.4, 112.4)
- added C34: CL10C060DB8NNNC, Capacitor_SMD:C_0603_1608Metric, F.Cu at (256.2, 112.1)
- added C35: CL05B104KA5NNNC, Capacitor_SMD:C_0402_1005Metric, F.Cu at (268.1, 111.8)
- added C36: CL21B475KAFNNNE, Capacitor_SMD:C_0805_2012Metric, F.Cu at (264.4, 115.4)
- added C37: CL10C060DB8NNNC, Capacitor_SMD:C_0603_1608Metric, F.Cu at (256.2, 114.6)
- added C38: CL21B475KAFNNNE, Capacitor_SMD:C_0805_2012Metric, F.Cu at (264.4, 118.4)
- added C39: CL21B475KAFNNNE, Capacitor_SMD:C_0805_2012Metric, F.Cu at (264.4, 121.4)
- added C4: CL21B106KQQNFNE, Capacitor_SMD:C_0805_2012Metric, F.Cu at (104.8, 58.8)
- added C40: CL21B475KAFNNNE, Capacitor_SMD:C_0805_2012Metric, F.Cu at (264.4, 124.4)
- added C41: CL05B104KA5NNNC, Capacitor_SMD:C_0402_1005Metric, F.Cu at (268.1, 113.8)
- added C42: CL05B104KA5NNNC, Capacitor_SMD:C_0402_1005Metric, F.Cu at (268.1, 115.8)
- added C43: CL05B104KA5NNNC, Capacitor_SMD:C_0402_1005Metric, F.Cu at (268.1, 117.8)
- added C44: CL05B104KA5NNNC, Capacitor_SMD:C_0402_1005Metric, F.Cu at (268.1, 119.7)
- added C45: CL05B104KA5NNNC, Capacitor_SMD:C_0402_1005Metric, F.Cu at (268.1, 121.7)
- added C46: GRM32EE70G107ME19K, Capacitor_SMD:C_1210_3225Metric, F.Cu at (127.5, 70.3)
- added C47: CL21B475KPFNNNE, Capacitor_SMD:C_0805_2012Metric, B.Cu at (133.1, 90.0)
- added C48: GRM32EE70G107ME19K, Capacitor_SMD:C_1210_3225Metric, F.Cu at (134.9, 91.5)
- added C49: GRM188R70J474KA01D, Capacitor_SMD:C_0603_1608Metric, B.Cu at (140.1, 92.9)
- added C5: CL21B106KQQNFNE, Capacitor_SMD:C_0805_2012Metric, F.Cu at (102.8, 58.8)
- added C50: CL21B475KPFNNNE, Capacitor_SMD:C_0805_2012Metric, B.Cu at (138.1, 83.5)
- added C51: GRM188R70J474KA01D, Capacitor_SMD:C_0603_1608Metric, B.Cu at (126.7, 87.3)
- added C52: GRM32EE70G107ME19K, Capacitor_SMD:C_1210_3225Metric, F.Cu at (132.3, 70.3)
- added C53: GRM188R70J474KA01D, Capacitor_SMD:C_0603_1608Metric, B.Cu at (137.9, 79.4)
- added C54: GRM32ER70J476ME20L, Capacitor_SMD:C_1210_3225Metric, F.Cu at (145.5, 39.0)
- added C55: GRM32EE70G107ME19K, Capacitor_SMD:C_1210_3225Metric, F.Cu at (137.1, 70.3)
- added C56: GRM32EE70G107ME19K, Capacitor_SMD:C_1210_3225Metric, F.Cu at (145.5, 47.5)
- added C57: GRM188R70J474KA01D, Capacitor_SMD:C_0603_1608Metric, B.Cu at (135.1, 93.0)
- added C58: CL21B475KPFNNNE, Capacitor_SMD:C_0805_2012Metric, F.Cu at (125.9, 44.5)
- added C59: CL21B475KPFNNNE, Capacitor_SMD:C_0805_2012Metric, B.Cu at (126.9, 57.9)
- added C6: CL05B102KB5NNNC, Capacitor_SMD:C_0402_1005Metric, F.Cu at (102.1, 54.5)
- added C60: GRM188R70J474KA01D, Capacitor_SMD:C_0603_1608Metric, B.Cu at (150.6, 60.6)
- added C61: CL21B475KPFNNNE, Capacitor_SMD:C_0805_2012Metric, B.Cu at (125.2, 98.1)
- added C62: CL21B475KPFNNNE, Capacitor_SMD:C_0805_2012Metric, F.Cu at (130.3, 38.4)
- added C63: GRM188R70J474KA01D, Capacitor_SMD:C_0603_1608Metric, B.Cu at (129.4, 89.7)
- added C64: GRM188R70J474KA01D, Capacitor_SMD:C_0603_1608Metric, F.Cu at (144.3, 34.6)
- added C65: GRM188R70J474KA01D, Capacitor_SMD:C_0603_1608Metric, B.Cu at (126.9, 59.9)
- added C66: GRM188R70J474KA01D, Capacitor_SMD:C_0603_1608Metric, B.Cu at (140.5, 70.5)
- added C67: GRM188R70J474KA01D, Capacitor_SMD:C_0603_1608Metric, B.Cu at (128.0, 70.1)
- added C68: GRM188R70J474KA01D, Capacitor_SMD:C_0603_1608Metric, F.Cu at (148.3, 27.1)
- added C69: GRM32ER70J476ME20L, Capacitor_SMD:C_1210_3225Metric, F.Cu at (151.2, 39.0)
- added C7: CL05B104KA5NNNC, Capacitor_SMD:C_0402_1005Metric, F.Cu at (212.2, 102.9)
- added C70: GRM32ER70J476ME20L, Capacitor_SMD:C_1210_3225Metric, F.Cu at (151.2, 43.3)
- added C71: GRM32ER70J476ME20L, Capacitor_SMD:C_1210_3225Metric, F.Cu at (151.2, 47.5)
- added C72: GRM32ER70J476ME20L, Capacitor_SMD:C_1210_3225Metric, F.Cu at (156.8, 39.0)
- added C73: GRM32EE70G107ME19K, Capacitor_SMD:C_1210_3225Metric, F.Cu at (156.8, 43.3)
- added C74: GRM32ER70J476ME20L, Capacitor_SMD:C_1210_3225Metric, F.Cu at (139.6, 55.5)
- added C75: CL21B475KPFNNNE, Capacitor_SMD:C_0805_2012Metric, F.Cu at (130.3, 41.4)
- added C76: CL21B475KPFNNNE, Capacitor_SMD:C_0805_2012Metric, F.Cu at (154.0, 156.7)
- added C77: CL10B105KA8NNNC, Capacitor_SMD:C_0603_1608Metric, F.Cu at (146.9, 149.2)
- added C78: CL10B105KA8NNNC, Capacitor_SMD:C_0603_1608Metric, F.Cu at (146.9, 151.7)
- added C79: CL05B104KA5NNNC, Capacitor_SMD:C_0402_1005Metric, F.Cu at (150.3, 156.2)
- added C8: CL05B104KA5NNNC, Capacitor_SMD:C_0402_1005Metric, F.Cu at (105.8, 49.6)
- added C80: CL05B103KB5NNNC, Capacitor_SMD:C_0402_1005Metric, F.Cu at (150.3, 158.2)
- added C81: CL05B104KA5NNNC, Capacitor_SMD:C_0402_1005Metric, F.Cu at (150.3, 160.1)
- added C82: CL21B475KPFNNNE, Capacitor_SMD:C_0805_2012Metric, F.Cu at (130.3, 44.5)
- added C83: CL21B475KPFNNNE, Capacitor_SMD:C_0805_2012Metric, F.Cu at (130.3, 47.5)
- added C84: CL21B475KPFNNNE, Capacitor_SMD:C_0805_2012Metric, F.Cu at (130.3, 50.5)
- added C85: CL21B475KPFNNNE, Capacitor_SMD:C_0805_2012Metric, F.Cu at (134.8, 38.4)
- added C86: GRM188R70J474KA01D, Capacitor_SMD:C_0603_1608Metric, F.Cu at (148.3, 29.6)
- added C87: CL21B475KPFNNNE, Capacitor_SMD:C_0805_2012Metric, F.Cu at (134.8, 41.4)
- added C88: CL21B475KPFNNNE, Capacitor_SMD:C_0805_2012Metric, F.Cu at (134.8, 44.5)
- added C89: CL21B475KPFNNNE, Capacitor_SMD:C_0805_2012Metric, F.Cu at (134.8, 47.5)
- added C9: CL21B106KQQNFNE, Capacitor_SMD:C_0805_2012Metric, F.Cu at (106.8, 58.8)
- added C90: GRM188R70J474KA01D, Capacitor_SMD:C_0603_1608Metric, F.Cu at (148.3, 32.1)
- added C91: GRM188R70J474KA01D, Capacitor_SMD:C_0603_1608Metric, F.Cu at (148.3, 34.6)
- added C92: GRM188R70J474KA01D, Capacitor_SMD:C_0603_1608Metric, F.Cu at (152.3, 19.5)
- added C93: GRM188R70J474KA01D, Capacitor_SMD:C_0603_1608Metric, F.Cu at (152.3, 22.0)
- added C94: GRM188R70J474KA01D, Capacitor_SMD:C_0603_1608Metric, F.Cu at (152.3, 24.6)
- added C95: GRM188R70J474KA01D, Capacitor_SMD:C_0603_1608Metric, F.Cu at (152.3, 27.1)
- added C96: GRM188R70J474KA01D, Capacitor_SMD:C_0603_1608Metric, F.Cu at (152.3, 29.6)
- added C97: GRM188R70J474KA01D, Capacitor_SMD:C_0603_1608Metric, F.Cu at (152.3, 32.1)
- added C98: GRM188R70J474KA01D, Capacitor_SMD:C_0603_1608Metric, F.Cu at (152.3, 34.6)
- added C99: GRM188R70J474KA01D, Capacitor_SMD:C_0603_1608Metric, F.Cu at (156.4, 19.5)
- added D1: 150060BS75000, LED_SMD:LED_0603_1608Metric, F.Cu at (65.6, 148.0)
- added D2: 150060BS75000, LED_SMD:LED_0603_1608Metric, F.Cu at (65.6, 150.6)
- added D3: ESD204DQAR, Diodes:USON-10, F.Cu at (207.4, 72.1)
- added D4: 150060BS75000, LED_SMD:LED_0603_1608Metric, F.Cu at (57.8, 151.7)
- added FB1: MPZ1608S601ATA00, Resistor_SMD:R_0603_1608Metric, F.Cu at (84.1, 152.6)
- added FB10: MPZ1608S601ATA00, Resistor_SMD:R_0603_1608Metric, F.Cu at (193.3, 57.6)
- added FB11: MPZ1608S601ATA00, Resistor_SMD:R_0603_1608Metric, F.Cu at (193.3, 60.2)
- added FB2: MPZ1608S601ATA00, Resistor_SMD:R_0603_1608Metric, F.Cu at (200.7, 91.7)
- added FB3: MPZ1608S601ATA00, Resistor_SMD:R_0603_1608Metric, F.Cu at (200.7, 94.2)
- added FB4: MPZ1608S601ATA00, Resistor_SMD:R_0603_1608Metric, F.Cu at (200.7, 96.8)
- added FB5: MPZ1608S601ATA00, Resistor_SMD:R_0603_1608Metric, F.Cu at (200.7, 99.3)
- added FB6: MPZ1608S601ATA00, Resistor_SMD:R_0603_1608Metric, F.Cu at (200.7, 101.8)
- added FB7: MPZ1608S601ATA00, Resistor_SMD:R_0603_1608Metric, F.Cu at (200.7, 104.3)
- added FB8: MPZ1608S601ATA00, Resistor_SMD:R_0603_1608Metric, F.Cu at (256.2, 117.1)
- added FB9: MPZ1608S601ATA00, Resistor_SMD:R_0603_1608Metric, F.Cu at (256.2, 119.6)
- added H1: MountingHole_Pad, MountingHole:MountingHole_2mm, F.Cu at (169.8, 92.0)
- added H2: MountingHole_Pad, MountingHole:MountingHole_2mm, F.Cu at (127.1, 118.3)
- added J1: TC2050, Connector:Tag-Connect_TC2050-IDC-NL_2x05_P1.27mm_Vertical, F.Cu at (62.5, 172.1)
- added J2: 1054550101, Connectors:1054550101, F.Cu at (103.0, 122.1)
- added J3: DF40C-80DP-0.4V(58), Connectors:DF40C-80DP-0.4V, B.Cu at (154.9, 93.8)
- added J4: DF40C-70DP-0.4V(51), Connectors:DF40C-70DP-0.4V, B.Cu at (166.1, 108.1)
- added J5: DF40C-80DP-0.4V(58), Connectors:DF40C-80DP-0.4V, B.Cu at (151.2, 115.2)
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Routing:
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- added copper zone on F.Cu, net +VIN_5V0
- added copper zone on F.Cu, net GND
- added copper zone on F.Cu, net Net-(L2-Pad1)
- added copper zone on F.Cu, net Net-(L3-Pad1)
- added copper zone on F.Cu, net Net-(L4-Pad1)
- added copper zone on F.Cu, net Net-(L5-Pad1)
Other:
- board size 80 x 68.9 mm -> 102.2 x 100 mm
- copper layers 2 -> 8

Commit message: added starage, usb sch; more design progress in sch;
Parts:
- removed the C14 at (77.0, 136.8)
- added C164: CL05B473KA5VPNC, Capacitor_SMD:C_0402_1005Metric, B.Cu at (116.0, 82.2)
- added C165: CL05B473KA5VPNC, Capacitor_SMD:C_0402_1005Metric, B.Cu at (116.2, 84.1)
- added C166: CL05B473KA5VPNC, Capacitor_SMD:C_0402_1005Metric, B.Cu at (111.9, 88.6)
- added C167: CL05B473KA5VPNC, Capacitor_SMD:C_0402_1005Metric, B.Cu at (115.5, 90.8)
- added C168: CL05B473KA5VPNC, Capacitor_SMD:C_0402_1005Metric, B.Cu at (110.0, 86.5)
- added C169: CL05B473KA5VPNC, Capacitor_SMD:C_0402_1005Metric, B.Cu at (117.1, 89.8)
- added C170: CL05B473KA5VPNC, Capacitor_SMD:C_0402_1005Metric, B.Cu at (113.8, 89.3)
- added C171: CL05B473KA5VPNC, Capacitor_SMD:C_0402_1005Metric, B.Cu at (104.8, 82.2)
- added C172: CL05B473KA5VPNC, Capacitor_SMD:C_0402_1005Metric, B.Cu at (107.2, 82.2)
- added C173: CL05B473KA5VPNC, Capacitor_SMD:C_0402_1005Metric, B.Cu at (110.9, 83.4)
- added C174: CL05B473KA5VPNC, Capacitor_SMD:C_0402_1005Metric, B.Cu at (109.5, 83.0)
- added C175: CL05B473KA5VPNC, Capacitor_SMD:C_0402_1005Metric, B.Cu at (113.6, 84.3)
- added C176: CL05B473KA5VPNC, Capacitor_SMD:C_0402_1005Metric, B.Cu at (114.2, 82.2)
- added C177: CL05B473KA5VPNC, Capacitor_SMD:C_0402_1005Metric, B.Cu at (112.8, 90.8)
- added C178: CL05B473KA5VPNC, Capacitor_SMD:C_0402_1005Metric, B.Cu at (110.9, 90.8)
- added C179: CL05B473KA5VPNC, Capacitor_SMD:C_0402_1005Metric, B.Cu at (112.3, 82.2)
- added C180: CL05B473KA5VPNC, Capacitor_SMD:C_0402_1005Metric, B.Cu at (104.7, 90.8)
- added C181: CL05B473KA5VPNC, Capacitor_SMD:C_0402_1005Metric, B.Cu at (106.5, 90.8)
- added C182: CL05B473KA5VPNC, Capacitor_SMD:C_0402_1005Metric, B.Cu at (108.8, 88.7)
- added C183: CL05B103KB5NNNC, Capacitor_SMD:C_0402_1005Metric, F.Cu at (192.0, 116.3)
- added C184: CL05B103KB5NNNC, Capacitor_SMD:C_0402_1005Metric, F.Cu at (192.0, 115.4)
- added C185: CL05B104KA5NNNC, Capacitor_SMD:C_0402_1005Metric, F.Cu at (39.3, 24.8)
- added C186: CL21B475KPFNNNE, Capacitor_SMD:C_0805_2012Metric, F.Cu at (55.9, 106.4)
- added C187: CL05B102KB5NNNC, Capacitor_SMD:C_0402_1005Metric, F.Cu at (59.5, 116.2)
- added C188: CL21B106KQQNFNE, Capacitor_SMD:C_0805_2012Metric, F.Cu at (55.9, 109.4)
- added C189: CL21B106KQQNFNE, Capacitor_SMD:C_0805_2012Metric, F.Cu at (55.9, 112.4)
- added C190: CL05B104KA5NNNC, Capacitor_SMD:C_0402_1005Metric, F.Cu at (59.5, 118.2)
- added C191: CL21B106KQQNFNE, Capacitor_SMD:C_0805_2012Metric, F.Cu at (55.9, 115.4)
- added C192: CL21B106KQQNFNE, Capacitor_SMD:C_0805_2012Metric, F.Cu at (55.9, 118.4)
- added C193: CL21B106KQQNFNE, Capacitor_SMD:C_0805_2012Metric, F.Cu at (55.9, 121.4)
- added C194: CL10B105KA8NNNC, Capacitor_SMD:C_0603_1608Metric_Pad1.08x0.95mm_HandSolder, F.Cu at (24.8, 93.5)
- added C195: CL05B104KA5NNNC, Capacitor_SMD:C_0402_1005Metric_Pad0.74x0.62mm_HandSolder, F.Cu at (48.9, 102.2)
- added C196: CL21B475KAFNNNE, Capacitor_SMD:C_0805_2012Metric_Pad1.18x1.45mm_HandSolder, F.Cu at (45.6, 93.7)
- added C197: CL21B475KAFNNNE, Capacitor_SMD:C_0805_2012Metric_Pad1.18x1.45mm_HandSolder, F.Cu at (45.6, 96.7)
- added C198: CL21B475KAFNNNE, Capacitor_SMD:C_0805_2012Metric_Pad1.18x1.45mm_HandSolder, F.Cu at (45.6, 99.8)
- added C199: CL21B475KAFNNNE, Capacitor_SMD:C_0805_2012Metric_Pad1.18x1.45mm_HandSolder, F.Cu at (29.1, 140.9)
- added C200: CL10B105KA8NNNC, Capacitor_SMD:C_0603_1608Metric_Pad1.08x0.95mm_HandSolder, F.Cu at (34.0, 136.1)
- added C201: CL05B104KA5NNNC, Capacitor_SMD:C_0402_1005Metric, F.Cu at (37.6, 135.8)
- added C202: CL05B104KA5NNNC, Capacitor_SMD:C_0402_1005Metric, F.Cu at (51.8, 134.0)
- added C203: CL05B104KA5NNNC, Capacitor_SMD:C_0402_1005Metric, F.Cu at (51.8, 135.9)
- added C204: CL05B104KA5NNNC, Capacitor_SMD:C_0402_1005Metric, F.Cu at (51.8, 137.9)
- added FB12: MPZ1608S601ATA00, Resistor_SMD:R_0603_1608Metric, F.Cu at (24.6, 129.4)
- added R123: RC0402FR-07240RL, Resistor_SMD:R_0402_1005Metric, F.Cu at (187.9, 107.0)
- added R124: RC0603FR-0710KL, Resistor_SMD:R_0603_1608Metric, F.Cu at (60.1, 111.5)
- added R125: RC0603FR-0710KL, Resistor_SMD:R_0603_1608Metric, F.Cu at (60.1, 114.0)
- added R126: RC0402FR-07100KL, Resistor_SMD:R_0402_1005Metric, F.Cu at (59.6, 120.2)
- added R127: RC0603FR-0747K5L, Resistor_SMD:R_0603_1608Metric_Pad0.98x0.95mm_HandSolder, F.Cu at (24.8, 96.0)
- added R128: RC0603FR-0747K5L, Resistor_SMD:R_0603_1608Metric_Pad0.98x0.95mm_HandSolder, F.Cu at (24.8, 98.5)
- added R129: RC0603FR-0747K5L, Resistor_SMD:R_0603_1608Metric_Pad0.98x0.95mm_HandSolder, F.Cu at (24.8, 101.0)
- added R130: RC0603FR-0710KL, Resistor_SMD:R_0603_1608Metric_Pad0.98x0.95mm_HandSolder, F.Cu at (24.8, 103.5)
- added R131: RC0402FR-0722RL, Resistor_SMD:R_0402_1005Metric, F.Cu at (48.7, 104.2)
- added R132: RC0603FR-0747K5L, Resistor_SMD:R_0603_1608Metric_Pad0.98x0.95mm_HandSolder, F.Cu at (24.8, 106.0)
- added R133: RC0603FR-0710KL, Resistor_SMD:R_0603_1608Metric_Pad0.98x0.95mm_HandSolder, F.Cu at (24.8, 108.5)
- added R134: RC0402FR-0722RL, Resistor_SMD:R_0603_1608Metric, F.Cu at (45.2, 105.0)
- added R137: RC0603FR-0710KL, Resistor_SMD:R_0603_1608Metric, F.Cu at (24.6, 137.0)
- added R138: RC0603FR-072KL, Resistor_SMD:R_0603_1608Metric_Pad0.98x0.95mm_HandSolder, F.Cu at (34.0, 138.6)
- added R139: RC0603FR-0710KL, Resistor_SMD:R_0603_1608Metric, F.Cu at (24.6, 139.5)
- added R140: RC0603FR-0710KL, Resistor_SMD:R_0603_1608Metric, F.Cu at (24.6, 142.0)
- added R141: RC0603FR-078K06L, Resistor_SMD:R_0603_1608Metric_Pad0.98x0.95mm_HandSolder, F.Cu at (48.2, 134.2)
- added R142: RC0603FR-0710KL, Resistor_SMD:R_0603_1608Metric, F.Cu at (44.0, 134.2)
- added R143: RC0402FR-07100RL, Resistor_SMD:R_0603_1608Metric, F.Cu at (44.0, 136.8)
- added R144: RC0402FR-07100RL, Resistor_SMD:R_0603_1608Metric, F.Cu at (44.0, 139.3)
- added R145: RC0603FR-071ML, Resistor_SMD:R_0603_1608Metric_Pad0.98x0.95mm_HandSolder, F.Cu at (48.2, 136.8)
- added U12: TPS51200DRCR, Package_SON:VSON-10-1EP_3x3mm_P0.5mm_EP1.65x2.4mm, F.Cu at (60.8, 107.5)
- added U13: S25FL128SAGNFI003, ICs:PG-WSON-8_EP, F.Cu at (46.8, 111.4)
- added U14: MX52LM04A11XSI, ICs:LFBGA-153_11.5x13mm_Layout14x14_P0.5mm, F.Cu at (34.3, 115.7)
- added U15: FT232HQ-REEL, Package_DFN_QFN:QFN-48-1EP_7x7mm_P0.5mm_EP5.1x5.1mm, F.Cu at (60.0, 130.3)
- added U16: 93LC56BT-I/OT, Package_TO_SOT_SMD:SOT-23-6, F.Cu at (29.2, 137.2)
- added U17: USB3320C-EZK, Package_DFN_QFN:QFN-32-1EP_5x5mm_P0.5mm_EP3.1x3.1mm, F.Cu at (45.6, 129.3)
- added U8: AS4C256M16D3C-12BCN, Package_BGA:BGA-96_9.0x13.0mm_Layout2x3x16_P0.8mm, F.Cu at (54.1, 21.8)
- added Y3: ECS-2033-250-BN, Miscellaneous:ECS-2033, F.Cu at (39.7, 21.8)
- added Y4: ECS-240-12-37B-CKY-TR, Miscellaneous:ECX-1637B, F.Cu at (51.3, 127.5)
- C121, C122, C123, C124, C125, C131, C132, C133, C134, C135, C141, C142, C143, C144, C145, C151, C152, C153, C154, J9: moved to F.Cu
- R100, R101, R102, R103, R104, R105, R106, R107, R108, R109, R110, R111, R112, R113, R114, R115, R116, R117, R118, R22, R23, R27, R28, R29, R30, R95, R96, R97, R98, R99: footprint Resistor_SMD:R_0402_1005Metric -> Resistor_SMD:R_0603_1608Metric
- Y1: footprint Miscellaneous:ECS-2033-500-BN -> Miscellaneous:ECS-2033
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Connections:
- net +VTT_REF renamed +PS_VTT_REF
- net /ST_I2C1_SCL renamed /mcu/ST_I2C1_SCL
- net /ST_I2C1_SDA renamed /mcu/ST_I2C1_SDA
- net /power/VTT_EN renamed /power/PS_VTT_EN
- net /power/VTT_PGOOD renamed /power/PS_VTT_PGOOD
- net /soc/soc-ddr/DDR3_A0 renamed /soc/soc-ram/DDR3_A0
- net /soc/soc-ddr/DDR3_A1 renamed /soc/soc-ram/DDR3_A1
- net /soc/soc-ddr/DDR3_A10 renamed /soc/soc-ram/DDR3_A10
- net /soc/soc-ddr/DDR3_A11 renamed /soc/soc-ram/DDR3_A11
- net /soc/soc-ddr/DDR3_A12 renamed /soc/soc-ram/DDR3_A12
- net /soc/soc-ddr/DDR3_A13 renamed /soc/soc-ram/DDR3_A13
- net /soc/soc-ddr/DDR3_A14 renamed /soc/soc-ram/DDR3_A14
- net /soc/soc-ddr/DDR3_A2 renamed /soc/soc-ram/DDR3_A2
- net /soc/soc-ddr/DDR3_A3 renamed /soc/soc-ram/DDR3_A3
- net /soc/soc-ddr/DDR3_A4 renamed /soc/soc-ram/DDR3_A4
- net /soc/soc-ddr/DDR3_A5 renamed /soc/soc-ram/DDR3_A5
- net /soc/soc-ddr/DDR3_A6 renamed /soc/soc-ram/DDR3_A6
- net /soc/soc-ddr/DDR3_A7 renamed /soc/soc-ram/DDR3_A7
- net /soc/soc-ddr/DDR3_A8 renamed /soc/soc-ram/DDR3_A8
- net /soc/soc-ddr/DDR3_A9 renamed /soc/soc-ram/DDR3_A9
- net /soc/soc-ddr/DDR3_ADDR0 renamed /soc/soc-ram/DDR3_ADDR0
- net /soc/soc-ddr/DDR3_ADDR1 renamed /soc/soc-ram/DDR3_ADDR1
- net /soc/soc-ddr/DDR3_ADDR10 renamed /soc/soc-ram/DDR3_ADDR10
- net /soc/soc-ddr/DDR3_ADDR11 renamed /soc/soc-ram/DDR3_ADDR11
- net /soc/soc-ddr/DDR3_ADDR12 renamed /soc/soc-ram/DDR3_ADDR12
- net /soc/soc-ddr/DDR3_ADDR13 renamed /soc/soc-ram/DDR3_ADDR13
- net /soc/soc-ddr/DDR3_ADDR14 renamed /soc/soc-ram/DDR3_ADDR14
- net /soc/soc-ddr/DDR3_ADDR2 renamed /soc/soc-ram/DDR3_ADDR2
- net /soc/soc-ddr/DDR3_ADDR3 renamed /soc/soc-ram/DDR3_ADDR3
- net /soc/soc-ddr/DDR3_ADDR4 renamed /soc/soc-ram/DDR3_ADDR4
- net /soc/soc-ddr/DDR3_ADDR5 renamed /soc/soc-ram/DDR3_ADDR5
- net /soc/soc-ddr/DDR3_ADDR6 renamed /soc/soc-ram/DDR3_ADDR6
- net /soc/soc-ddr/DDR3_ADDR7 renamed /soc/soc-ram/DDR3_ADDR7
- net /soc/soc-ddr/DDR3_ADDR8 renamed /soc/soc-ram/DDR3_ADDR8
- net /soc/soc-ddr/DDR3_ADDR9 renamed /soc/soc-ram/DDR3_ADDR9
- net /soc/soc-ddr/DDR3_CK+ renamed /soc/soc-ram/DDR3_CK+
- net /soc/soc-ddr/DDR3_CK- renamed /soc/soc-ram/DDR3_CK-
- net /soc/soc-ps/MODE0 renamed /soc/FLSH_QSPI_IO3
- net /soc/soc-ps/MODE1 renamed /soc/FLSH_QSPI_IO1
- net /soc/soc-ps/MODE2 renamed /soc/FLSH_QSPI_IO2
- net /soc/soc-ps/MODE3 renamed /soc/FLSH_QSPI_IO0
- net /soc/soc-ps/MODE4 renamed /soc/FLSH_QSPI_SCK
- net /soc/soc-ps/SD_CLK renamed /soc/SD_CLK
- net /soc/soc-ps/SD_CMD renamed /soc/SD_CMD
- net /soc/soc-ps/SD_D0 renamed /soc/SD_D0
- net /soc/soc-ps/SD_D1 renamed /soc/SD_D1
- net /soc/soc-ps/SD_D2 renamed /soc/SD_D2
- net /soc/soc-ps/SD_D3 renamed /soc/SD_D3
- net /soc/soc-ps/SD_SEL renamed /soc/SD_SEL
- net /soc/soc-ps/VCFG0 renamed /soc/soc-ps/MIO7
- net /soc/soc-ps/VCFG1 renamed /soc/soc-ps/MIO8
- net Net-(D4-A) renamed /soc/soc-ps/ZYNQ_DONE_0
- net Net-(J9-CLK) renamed /soc/SDC_CLK
- net Net-(J9-CMD) renamed /soc/SDC_CMD
- net Net-(J9-DAT0) renamed /soc/SDC_DAT0
- net Net-(J9-DAT1) renamed /soc/SDC_DAT1
- net Net-(J9-DAT2) renamed /soc/SDC_DAT2
- net Net-(J9-DAT3) renamed /soc/SDC_DAT3
- C10 pad 1: +VTT_0V75 -> +PS_VTT_0V75
- C11 pad 1: +VTT_0V75 -> +PS_VTT_0V75
- C111 pad 1: +VTT_0V75 -> +PS_VTT_0V75
- C112 pad 1: +VTT_0V75 -> +PS_VTT_0V75
- C113 pad 1: +VTT_0V75 -> +PS_VTT_0V75
- C114 pad 1: +VTT_0V75 -> +PS_VTT_0V75
- C115 pad 1: +VTT_0V75 -> +PS_VTT_0V75
- C116 pad 1: +VTT_0V75 -> +PS_VTT_0V75
- C117 pad 1: +VTT_0V75 -> +PS_VTT_0V75
- C118 pad 1: +VTT_0V75 -> +PS_VTT_0V75
- C119 pad 1: +VTT_0V75 -> +PS_VTT_0V75
- C120 pad 1: +VTT_0V75 -> +PS_VTT_0V75
- C4 pad 1: +VCC_1V5 -> +PS_VCC_1V5
- C5 pad 1: +VCC_1V5 -> +PS_VCC_1V5
- C9 pad 1: +VTT_0V75 -> +PS_VTT_0V75
- D3 pad 10: Net-(D3-NC-Pad10) -> /soc/soc-ps/JTAG_TDO
- D3 pad 6: Net-(D3-NC-Pad6) -> /soc/soc-ps/JTAG_TMS
- D3 pad 7: Net-(D3-NC-Pad7) -> /soc/soc-ps/JTAG_TCK
- D3 pad 9: Net-(D3-NC-Pad9) -> /soc/soc-ps/JTAG_TDI
- J2 pad A1: GND -> GND_USB
- J2 pad A10: unconnected-(J2-RX2--PadA10) -> /ftdi/USBC_RX2-N
- J2 pad A11: unconnected-(J2-RX2+-PadA11) -> /ftdi/USBC_RX2-P
- J2 pad A12: GND -> GND_USB
- J2 pad A2: unconnected-(J2-TX1+-PadA2) -> /ftdi/USBC_TX1-P
- J2 pad A3: unconnected-(J2-TX1--PadA3) -> /ftdi/USBC_TX1-N
- J2 pad A6: /USBC_D+ -> /ftdi/FTDI_USB_D+
- J2 pad A7: /USBC_D- -> /ftdi/FTDI_USB_D-
- J2 pad B1: GND -> GND_USB
- J2 pad B10: unconnected-(J2-RX1--PadB10) -> /ftdi/USBC_RX1-N
- J2 pad B11: unconnected-(J2-RX1+-PadB11) -> /ftdi/USBC_RX1-P
- J2 pad B12: GND -> GND_USB
- J2 pad B2: unconnected-(J2-TX2+-PadB2) -> /ftdi/USBC_TX2-P
- J2 pad B3: unconnected-(J2-TX2--PadB3) -> /ftdi/USBC_TX2-N
- J2 pad B6: /USBC_D+ -> /ftdi/FTDI_USB_D+
- J2 pad B7: /USBC_D- -> /ftdi/FTDI_USB_D-
- J2 pad SH1: GND -> GND_USB
- J2 pad SH2: GND -> GND_USB
- J7 pad 1: Net-(J9-CD) -> /soc/soc-ps/SD0_CD
- J7 pad 2: /soc/soc-ps/SD_CD -> /soc/SDC_CD
- J8 pad 2: /soc/soc-ps/SD_CD -> /soc/soc-ps/SD0_CD
- J9 pad 9: Net-(J9-CD) -> /soc/SDC_CD
- R1 pad 1: +VCC_1V5 -> +PS_VCC_1V5
- R10 pad 2: +VCC_1V5 -> +PS_VCC_1V5
- R110 pad 1: /soc/soc-ddr/DDR3_BA2 -> /soc/soc-ram/DDR3_BA2
- R111 pad 1: /soc/soc-ddr/DDR3_BA1 -> /soc/soc-ram/DDR3_BA1
- R112 pad 1: /soc/soc-ddr/DDR3_BA0 -> /soc/soc-ram/DDR3_BA0
- R113 pad 1: /soc/soc-ddr/DDR3_RAS -> /soc/soc-ram/DDR3_nRAS
- R114 pad 1: /soc/soc-ddr/DDR3_CAS -> /soc/soc-ram/DDR3_nCAS
- R115 pad 1: /soc/soc-ddr/DDR3_CS -> /soc/soc-ram/DDR3_nCS
- R116 pad 1: /soc/soc-ddr/DDR3_WE -> /soc/soc-ram/DDR3_nWE
- R117 pad 1: /soc/soc-ddr/DDR3_CKE -> /soc/soc-ram/DDR3_CKE
- R118 pad 1: /soc/soc-ddr/DDR3_ODT0 -> /soc/soc-ram/DDR3_ODT0
- R118 pad 2: Net-(U5F-PS_DDR_ODT_502) -> unconnected-(R118-Pad2)
- R120 pad 1: Net-(U5F-PS_DDR_VRN_502) -> unconnected-(R120-Pad1)
- R120 pad 2: +VCC_1V5 -> +PS_VCC_1V5
- R121 pad 1: Net-(U9-ZQ) -> Net-(U8-ZQ)
- R21 pad 1: Net-(Y1-OUT) -> Net-(Y3-OUT)
- R45 pad 1: Net-(D3-NC-Pad10) -> /soc/soc-ps/JTAG_TDO
- R46 pad 1: Net-(D3-NC-Pad9) -> /soc/soc-ps/JTAG_TDI
- R47 pad 1: Net-(D3-NC-Pad7) -> /soc/soc-ps/JTAG_TCK
- R48 pad 1: Net-(D3-NC-Pad6) -> /soc/soc-ps/JTAG_TMS
- R52 pad 2: /soc/soc-ps/SD_CD -> /soc/SDC_CD
- R6 pad 2: GND -> GND_USB
- R68 pad 1: +VTT_0V75 -> +PS_VTT_0V75
- R68 pad 2: /soc/soc-ddr/DDR_ODT0 -> /soc/soc-ram/DDR3_ODT0
- R69 pad 1: +VTT_0V75 -> +PS_VTT_0V75
- R69 pad 2: /soc/soc-ddr/DDR_nWE -> /soc/soc-ram/DDR3_nWE
- R7 pad 2: GND -> GND_USB
- R70 pad 1: +VTT_0V75 -> +PS_VTT_0V75
- R70 pad 2: /soc/soc-ddr/DDR_nCAS -> /soc/soc-ram/DDR3_nCAS
- R71 pad 1: +VTT_0V75 -> +PS_VTT_0V75
- R71 pad 2: /soc/soc-ddr/DDR_nRAS -> /soc/soc-ram/DDR3_nRAS
- R72 pad 1: +VTT_0V75 -> +PS_VTT_0V75
- R72 pad 2: /soc/soc-ddr/DDR_nCS -> /soc/soc-ram/DDR3_nCS
- R73 pad 1: +VTT_0V75 -> +PS_VTT_0V75
- R73 pad 2: /soc/soc-ddr/DDR_CKE -> /soc/soc-ram/DDR3_CKE
- R74 pad 1: +VTT_0V75 -> +PS_VTT_0V75
- R74 pad 2: /soc/soc-ddr/DDR_BA2 -> /soc/soc-ram/DDR3_BA2
- R75 pad 1: +VTT_0V75 -> +PS_VTT_0V75
- R75 pad 2: /soc/soc-ddr/DDR_BA1 -> /soc/soc-ram/DDR3_BA1
- R76 pad 1: +VTT_0V75 -> +PS_VTT_0V75
- R76 pad 2: /soc/soc-ddr/DDR_BA0 -> /soc/soc-ram/DDR3_BA0
- R77 pad 1: +VTT_0V75 -> +PS_VTT_0V75
- R78 pad 1: +VTT_0V75 -> +PS_VTT_0V75
- R79 pad 1: +VTT_0V75 -> +PS_VTT_0V75
- R80 pad 1: +VTT_0V75 -> +PS_VTT_0V75
- R81 pad 1: +VTT_0V75 -> +PS_VTT_0V75
- R82 pad 1: +VTT_0V75 -> +PS_VTT_0V75
- R83 pad 1: +VTT_0V75 -> +PS_VTT_0V75
- R84 pad 1: +VTT_0V75 -> +PS_VTT_0V75
- R85 pad 1: +VTT_0V75 -> +PS_VTT_0V75
- R86 pad 1: +VTT_0V75 -> +PS_VTT_0V75
- R87 pad 1: +VTT_0V75 -> +PS_VTT_0V75
- R88 pad 1: +VTT_0V75 -> +PS_VTT_0V75
- R89 pad 1: +VTT_0V75 -> +PS_VTT_0V75
- R90 pad 1: +VTT_0V75 -> +PS_VTT_0V75
- R91 pad 1: +VTT_0V75 -> +PS_VTT_0V75
- R92 pad 1: /soc/soc-ddr/DDR3_RST -> /soc/soc-ram/DDR3_RST
- R93 pad 1: +VCC_1V5 -> +PS_VCC_1V5
- R93 pad 2: /soc/soc-ddr/DDR3_CKE -> /soc/soc-ram/DDR3_CKE
- R94 pad 1: Net-(U5F-PS_DDR_VRP_502) -> unconnected-(R94-Pad1)
- U11 pad A2: /soc/soc-ddr/DDR3_D29 -> /soc/soc-ram/DDR3_D13
- U11 pad A3: /soc/soc-ddr/DDR3_D31 -> /soc/soc-ram/DDR3_D15
- U11 pad A7: /soc/soc-ddr/DDR3_D28 -> /soc/soc-ram/DDR3_D12
- U11 pad B7: /soc/soc-ddr/DDR3_DQS3- -> /soc/soc-ram/DDR3_DQS1-
- U11 pad B8: /soc/soc-ddr/DDR3_D30 -> /soc/soc-ram/DDR3_D14
- U11 pad C2: /soc/soc-ddr/DDR3_D27 -> /soc/soc-ram/DDR3_D11
- U11 pad C3: /soc/soc-ddr/DDR3_D25 -> /soc/soc-ram/DDR3_D9
- U11 pad C7: /soc/soc-ddr/DDR3_DQS3+ -> /soc/soc-ram/DDR3_DQS1+
- U11 pad C8: /soc/soc-ddr/DDR3_D26 -> /soc/soc-ram/DDR3_D10
- U11 pad D3: /soc/soc-ddr/DDR3_DM3 -> /soc/soc-ram/DDR3_DM1
- U11 pad D7: /soc/soc-ddr/DDR3_D24 -> /soc/soc-ram/DDR3_D8
- U11 pad E3: /soc/soc-ddr/DDR3_D16 -> /soc/soc-ram/DDR3_D0
- U11 pad E7: /soc/soc-ddr/DDR3_DM2 -> /soc/soc-ram/DDR3_DM0
- U11 pad F2: /soc/soc-ddr/DDR3_D18 -> /soc/soc-ram/DDR3_D2
- U11 pad F3: /soc/soc-ddr/DDR3_DQS2+ -> /soc/soc-ram/DDR3_DQS0+
- U11 pad F7: /soc/soc-ddr/DDR3_D17 -> /soc/soc-ram/DDR3_D1
- U11 pad F8: /soc/soc-ddr/DDR3_D19 -> /soc/soc-ram/DDR3_D3
- U11 pad G2: /soc/soc-ddr/DDR3_D22 -> /soc/soc-ram/DDR3_D6
- U11 pad G3: /soc/soc-ddr/DDR3_DQS2- -> /soc/soc-ram/DDR3_DQS0-
- U11 pad H3: /soc/soc-ddr/DDR3_D20 -> /soc/soc-ram/DDR3_D4
- U11 pad H7: /soc/soc-ddr/DDR3_D23 -> /soc/soc-ram/DDR3_D7
- U11 pad H8: /soc/soc-ddr/DDR3_D21 -> /soc/soc-ram/DDR3_D5
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Routing:
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Other:
- copper layers 8 -> 10

Commit message: routing changes; added mezzanine; added pl ram;
Parts:
- removed J3, J5: DF40C-80DP-0.4V(58), Connectors:DF40C-80DP-0.4V
- removed J4: DF40C-70DP-0.4V(51), Connectors:DF40C-70DP-0.4V
- added C205: CL31A106KBHNNNE, Capacitor_SMD:C_1206_3216Metric, B.Cu at (176.9, 102.7)
- added C206: CL05B104KA5NNNC, Capacitor_SMD:C_0402_1005Metric, B.Cu at (175.1, 104.0)
- added C207: CL05B104KA5NNNC, Capacitor_SMD:C_0402_1005Metric, B.Cu at (168.6, 99.5)
- added C208: CL05B104KA5NNNC, Capacitor_SMD:C_0402_1005Metric, B.Cu at (161.5, 106.5)
- added C209: CL05B104KA5NNNC, Capacitor_SMD:C_0402_1005Metric, B.Cu at (173.8, 104.0)
- added C210: CL10C060DB8NNNC, Capacitor_SMD:C_0603_1608Metric, F.Cu at (163.4, 80.7)
- added C211: CL10C060DB8NNNC, Capacitor_SMD:C_0603_1608Metric, F.Cu at (166.5, 80.7)
- C151: value CL05B473KA5VPNC -> CL05B103KB5NNNC
- C159: value CL05B103KB5NNNC -> CL05B473KA5VPNC
- C16, C17, C185, C19, C195, C196, C197, C198, C20, C21, C22, C23, C24, C25, C26, C27, C28, C29, C30, C31, C32, C7, C76, C77, C78, C79, C80, C81, FB2, FB3, FB4, FB5, FB6, FB7, R21, R24, R25, R26, R34, U10, U6, Y1, Y3: moved to B.Cu
- J2: value 1054550101 -> 2216100001; footprint Connectors:1054550101 -> Connectors:2216100001
- R100, R101, R102, R103, R104, R105, R106, R107, R108, R109, R110, R111, R112, R113, R114, R115, R116, R117, R118, R134, R95, R96, R97, R98, R99: footprint Resistor_SMD:R_0603_1608Metric -> Resistor_SMD:R_0402_1005Metric_Pad0.72x0.64mm_HandSolder
- R131: footprint Resistor_SMD:R_0402_1005Metric -> Resistor_SMD:R_0402_1005Metric_Pad0.72x0.64mm_HandSolder
- R22, R23, R27, R28, R29, R30: footprint Resistor_SMD:R_0603_1608Metric -> Resistor_SMD:R_0402_1005Metric_Pad0.72x0.64mm_HandSolder; moved to B.Cu
- moved R138 251.0 mm to (284.5, 123.1)
- moved U16 251.0 mm to (279.8, 121.8)
- moved C201 251.0 mm to (288.1, 120.4)
- moved R137 251.0 mm to (275.2, 121.5)
- moved R139 251.0 mm to (275.2, 124.1)
- moved R140 251.0 mm to (275.2, 126.6)
- moved C185 166.0 mm to (181.0, 111.2), turned to -90 degrees
- moved Y3 165.5 mm to (178.8, 111.6), turned to 180 degrees
- moved R145 142.0 mm to (180.6, 85.5), turned to 90 degrees
- moved C204 141.6 mm to (181.8, 81.9), turned to 90 degrees
- moved R142 141.3 mm to (178.1, 89.7), turned to 90 degrees
- moved Y2 141.0 mm to (130.6, 117.9), turned to 180 degrees
- moved C203 139.0 mm to (179.8, 81.9), turned to 90 degrees
- moved R141 138.8 mm to (178.1, 85.5), turned to 90 degrees
- moved Y1 137.6 mm to (164.6, 83.6)
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Connections:
- net /power/PL_VTT_EN renamed /soc/soc-pl/ram-pl/PL_VTT_EN
- net /power/PL_VTT_PGOOD renamed /soc/soc-pl/ram-pl/PL_VTT_PGOOD
- C151 pad 1: +VCC_1V5 -> +PL_VCC_1V5
- C160 pad 1: +VTT_0V75 -> +PL_VTT_0V75
- U5 pad A4: /soc/soc-ram/DDR3_D3 -> /soc/soc-ram/DDR3_D6
- U5 pad B3: /soc/soc-ram/DDR3_D1 -> /soc/soc-ram/DDR3_D0
- U5 pad C1: /soc/soc-ram/DDR3_D6 -> /soc/soc-ram/DDR3_D5
- U5 pad C3: /soc/soc-ram/DDR3_D0 -> /soc/soc-ram/DDR3_D4
- U5 pad D1: /soc/soc-ram/DDR3_D5 -> /soc/soc-ram/DDR3_D1
- U5 pad D18: unconnected-(U5C-IO_L3N_T0_DQS_AD1N_35-PadD18) -> /soc/soc-pl/AD1-
- U5 pad D3: /soc/soc-ram/DDR3_D4 -> /soc/soc-ram/DDR3_D7
- U5 pad E1: /soc/soc-ram/DDR3_D7 -> /soc/soc-ram/DDR3_D3
- U5 pad E17: unconnected-(U5C-IO_L3P_T0_DQS_AD1P_35-PadE17) -> /soc/soc-pl/AD1+
- U5 pad E18: unconnected-(U5C-IO_L5P_T0_AD9P_35-PadE18) -> /soc/soc-pl/AD9+
- U5 pad E19: unconnected-(U5C-IO_L5N_T0_AD9N_35-PadE19) -> /soc/soc-pl/AD9-
- U5 pad E2: /soc/soc-ram/DDR3_D8 -> /soc/soc-ram/DDR3_D15
- U5 pad E3: /soc/soc-ram/DDR3_D9 -> /soc/soc-ram/DDR3_D13
- U5 pad G19: unconnected-(U5C-IO_L18P_T2_AD13P_35-PadG19) -> /soc/soc-pl/AD13+
- U5 pad G20: unconnected-(U5C-IO_L18N_T2_AD13N_35-PadG20) -> /soc/soc-pl/AD13-
- U5 pad G3: /soc/soc-ram/DDR3_D10 -> /soc/soc-ram/DDR3_D11
- U5 pad H2: /soc/soc-ram/DDR3_D13 -> /soc/soc-ram/DDR3_D8
- U5 pad H20: unconnected-(U5C-IO_L17N_T2_AD5N_35-PadH20) -> /soc/soc-pl/AD5-
- U5 pad H3: /soc/soc-ram/DDR3_D11 -> /soc/soc-ram/DDR3_D9
- U5 pad J1: /soc/soc-ram/DDR3_D15 -> /soc/soc-ram/DDR3_D10
- U5 pad J14: unconnected-(U5C-IO_L20N_T3_AD6N_35-PadJ14) -> /soc/soc-pl/AD6-
- U5 pad J16: unconnected-(U5C-IO_L24N_T3_AD15N_35-PadJ16) -> /soc/soc-pl/AD15-
- U5 pad J19: unconnected-(U5C-IO_L10N_T1_AD11N_35-PadJ19) -> /soc/soc-pl/AD11-
- U5 pad J20: unconnected-(U5C-IO_L17P_T2_AD5P_35-PadJ20) -> /soc/soc-pl/AD5+
- U5 pad K14: unconnected-(U5C-IO_L20P_T3_AD6P_35-PadK14) -> /soc/soc-pl/AD6+
- U5 pad K16: unconnected-(U5C-IO_L24P_T3_AD15P_35-PadK16) -> /soc/soc-pl/AD15+
- U5 pad K19: unconnected-(U5C-IO_L10P_T1_AD11P_35-PadK19) -> /soc/soc-pl/AD11+
- U5 pad L14: unconnected-(U5C-IO_L22P_T3_AD7P_35-PadL14) -> /soc/soc-pl/AD7+
- U5 pad L15: unconnected-(U5C-IO_L22N_T3_AD7N_35-PadL15) -> /soc/soc-pl/AD7-
- U5 pad L19: unconnected-(U5C-IO_L9P_T1_DQS_AD3P_35-PadL19) -> /soc/soc-pl/AD3+
- U5 pad L20: unconnected-(U5C-IO_L9N_T1_DQS_AD3N_35-PadL20) -> /soc/soc-pl/AD3-
- U5 pad M17: unconnected-(U5C-IO_L8P_T1_AD10P_35-PadM17) -> /soc/soc-pl/AD10+
- U5 pad M18: unconnected-(U5C-IO_L8N_T1_AD10N_35-PadM18) -> /soc/soc-pl/AD10-
- U5 pad M19: unconnected-(U5C-IO_L7P_T1_AD2P_35-PadM19) -> /soc/soc-pl/AD2+
- U5 pad M20: unconnected-(U5C-IO_L7N_T1_AD2N_35-PadM20) -> /soc/soc-pl/AD2-
- U5 pad N15: unconnected-(U5C-IO_L21P_T3_DQS_AD14P_35-PadN15) -> /soc/soc-pl/AD14+
- U5 pad N16: unconnected-(U5C-IO_L21N_T3_DQS_AD14N_35-PadN16) -> /soc/soc-pl/AD14-
- U5 pad P1: /soc/soc-ram/DDR3_D16 -> /soc/soc-ram/DDR3_D18
- U5 pad P3: /soc/soc-ram/DDR3_D17 -> /soc/soc-ram/DDR3_D20
- U5 pad R1: /soc/soc-ram/DDR3_D19 -> /soc/soc-ram/DDR3_D16
- U5 pad R3: /soc/soc-ram/DDR3_D18 -> /soc/soc-ram/DDR3_D22
- U5 pad T4: /soc/soc-ram/DDR3_D20 -> /soc/soc-ram/DDR3_D23
- U5 pad U2: /soc/soc-ram/DDR3_D22 -> /soc/soc-ram/DDR3_D17
- U5 pad U3: /soc/soc-ram/DDR3_D23 -> /soc/soc-ram/DDR3_D19
- U5 pad V1: /soc/soc-ram/DDR3_D24 -> /soc/soc-ram/DDR3_D29
- U5 pad V2: /soc/soc-ram/DDR3_D30 -> /soc/soc-ram/DDR3_D31
- U5 pad V3: /soc/soc-ram/DDR3_D31 -> /soc/soc-ram/DDR3_D25
- U5 pad W1: /soc/soc-ram/DDR3_D26 -> /soc/soc-ram/DDR3_D27
- U5 pad W3: /soc/soc-ram/DDR3_D29 -> /soc/soc-ram/DDR3_D28
- U5 pad Y2: /soc/soc-ram/DDR3_D28 -> /soc/soc-ram/DDR3_D30
- U5 pad Y3: /soc/soc-ram/DDR3_D25 -> /soc/soc-ram/DDR3_D24
- U5 pad Y4: /soc/soc-ram/DDR3_D27 -> /soc/soc-ram/DDR3_D26
- U6 pad 4: +ETH_AVDDH -> +ETH_AVDDL
- U6 pad 9: +ETH_AVDDH -> +ETH_AVDDL
- U8 pad A1: +VCC_1V5 -> +PL_VCC_1V5
- U8 pad A8: +VCC_1V5 -> +PL_VCC_1V5
- U8 pad B2: +VCC_1V5 -> +PL_VCC_1V5
- U8 pad C1: +VCC_1V5 -> +PL_VCC_1V5
- U8 pad C9: +VCC_1V5 -> +PL_VCC_1V5
- U8 pad D2: +VCC_1V5 -> +PL_VCC_1V5
- U8 pad D9: +VCC_1V5 -> +PL_VCC_1V5
- U8 pad E9: +VCC_1V5 -> +PL_VCC_1V5
- U8 pad F1: +VCC_1V5 -> +PL_VCC_1V5
- U8 pad G7: +VCC_1V5 -> +PL_VCC_1V5
- U8 pad H1: +VTT_0V75 -> +PL_VTT_0V75
- U8 pad H2: +VCC_1V5 -> +PL_VCC_1V5
- U8 pad H9: +VCC_1V5 -> +PL_VCC_1V5
- U8 pad K2: +VCC_1V5 -> +PL_VCC_1V5
- U8 pad K8: +VCC_1V5 -> +PL_VCC_1V5
- U8 pad M8: +VTT_0V75 -> +PL_VTT_0V75
- U8 pad N1: +VCC_1V5 -> +PL_VCC_1V5
- U8 pad N9: +VCC_1V5 -> +PL_VCC_1V5
- U8 pad R1: +VCC_1V5 -> +PL_VCC_1V5
- U8 pad R9: +VCC_1V5 -> +PL_VCC_1V5
Routing:
- net (no net): track 131.1 -> 0.00 mm, vias 14 -> 0
- net /soc/soc-ram/DDR3_ADDR3: track 0.00 -> 25.8 mm
- net /soc/soc-ram/DDR3_ADDR0: track 0.00 -> 25.5 mm
- net /soc/soc-ram/DDR3_D6: track 0.00 -> 23.8 mm, vias 0 -> 2
- net /soc/soc-ram/DDR3_ADDR5: track 0.00 -> 23.8 mm
- net /soc/soc-ram/DDR3_D20: track 0.00 -> 23.7 mm, vias 0 -> 2
- net /soc/soc-ram/DDR3_D7: track 0.00 -> 23.6 mm, vias 0 -> 2
- net /soc/soc-ram/DDR3_D23: track 0.00 -> 23.3 mm, vias 0 -> 2
- net /soc/soc-ram/DDR3_D21: track 0.00 -> 23.2 mm, vias 0 -> 2
- net /soc/soc-ram/DDR3_ADDR2: track 0.00 -> 23.0 mm
- net /soc/soc-ps/USB0_DATA5: track 0.00 -> 22.3 mm, vias 0 -> 2
- net /soc/soc-ram/DDR3_D4: track 0.00 -> 22.1 mm, vias 0 -> 2
- net /soc/soc-ram/DDR3_DQS3+: track 0.00 -> 22.0 mm
- net /soc/soc-ram/DDR3_D5: track 0.00 -> 21.9 mm, vias 0 -> 2
- net /soc/soc-ps/USB0_DATA7: track 0.00 -> 21.8 mm, vias 0 -> 2
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Other:
- outline, holes or cut-outs redrawn
