File: Hardware/Design Files/rfsom-01/rfsom-01.kicad_pcb (KiCad board)
At the start: 10 copper layers, 102.2 x 100 mm, 411 parts, among them J1 TC2050, J2 2216100001, J9 DM3CS-SF, U1 TPS62086RLT, U10 STM32L432KCUx, U11 AS4C256M16D3C-12BCN, U12 TPS51200DRCR, U13 S25FL128SAGNFI003, U14 MX52LM04A11XSI, U15 FT232HQ-REEL, U16 93LC56BT-I/OT, U17 USB3320C-EZK, U2 TPS51200DRCR, U3 LP8758A1E0YFFR, U4 FT232HQ-REEL, U5 XC7Z010-1CLG400C, U6 KSZ9131RNXI-TR, U7 TXS02612RTWR, U8 AS4C256M16D3C-12BCN, U9 AS4C256M16D3C-12BCN, Y1 ECS-2033-500-BN, Y2 ABM10-166-12.000MHZ-T3, Y3 ECS-2033-250-BN, Y4 ECS-240-12-37B-CKY-TR

Commit message: updated sch pdf; routign progress;
Parts:
- removed U15: FT232HQ-REEL, Package_DFN_QFN:QFN-48-1EP_7x7mm_P0.5mm_EP5.1x5.1mm
- added C10: CL31A106KBHNNNE, Capacitor_SMD:C_1206_3216Metric_Pad1.33x1.80mm_HandSolder, F.Cu at (248.0, 73.7)
- added C11: CL31A106KBHNNNE, Capacitor_SMD:C_1206_3216Metric_Pad1.33x1.80mm_HandSolder, F.Cu at (248.0, 84.3)
- added C12: CL21B475KPFNNNE, Capacitor_SMD:C_0805_2012Metric, F.Cu at (224.9, 71.4)
- added C13: CL21B475KPFNNNE, Capacitor_SMD:C_0805_2012Metric, F.Cu at (224.9, 86.7)
- added C14: CL21B475KPFNNNE, Capacitor_SMD:C_0805_2012Metric, F.Cu at (248.0, 71.3)
- added C15: CL21B475KPFNNNE, Capacitor_SMD:C_0805_2012Metric, F.Cu at (248.0, 86.7)
- added C212: CL10B104KB8NNWC, Capacitor_SMD:C_0603_1608Metric_Pad1.08x0.95mm_HandSolder, F.Cu at (224.9, 69.5)
- added C213: CL10B104KB8NNWC, Capacitor_SMD:C_0603_1608Metric_Pad1.08x0.95mm_HandSolder, F.Cu at (224.9, 88.6)
- added C214: CL10B104KB8NNWC, Capacitor_SMD:C_0603_1608Metric_Pad1.08x0.95mm_HandSolder, F.Cu at (248.0, 69.3)
- added C215: CL10B104KB8NNWC, Capacitor_SMD:C_0603_1608Metric_Pad1.08x0.95mm_HandSolder, F.Cu at (248.0, 88.7)
- added C8: CL31A106KBHNNNE, Capacitor_SMD:C_1206_3216Metric_Pad1.33x1.80mm_HandSolder, F.Cu at (224.9, 73.8)
- added C9: CL31A106KBHNNNE, Capacitor_SMD:C_1206_3216Metric_Pad1.33x1.80mm_HandSolder, F.Cu at (224.9, 84.3)
- added J10: SEAM-40-02.0-L-04-2-A-K-TR, Connectors:SEAM-40-XX.X-XXX-04-X-A-XX-XX, B.Cu at (144.4, 74.0)
- added J3: SEAM-40-02.0-L-04-2-A-K-TR, Connectors:SEAM-40-XX.X-XXX-04-X-A-XX-XX, B.Cu at (145.3, 123.3)
- C16, C17, C185, C19, C20, C205, C206, C207, C208, C209, C21, C22, C23, C24, C25, C26, C27, C28, C29, C30, C31, C32, FB2, FB3, FB4, FB5, FB6, FB7, R21, R22, R23, R27, R28, R29, R30, R34, U6, Y3: moved to F.Cu
- J2, J9, R55, R56, R57, S2: moved to B.Cu
- moved L5 178.3 mm to (245.3, 81.4), turned to 0 degrees
- moved L4 175.6 mm to (245.3, 76.8), turned to 0 degrees
- moved C3 173.9 mm to (241.8, 81.4), turned to 90 degrees
- moved C5 171.1 mm to (241.8, 76.8), turned to 90 degrees
- moved R8 168.6 mm to (249.0, 76.8)
- moved R9 168.4 mm to (249.0, 81.4)
- moved U2 165.7 mm to (236.5, 79.1), turned to 90 degrees
- moved C2 160.6 mm to (231.2, 81.4), turned to 90 degrees
- moved C4 157.6 mm to (231.2, 76.8), turned to 90 degrees
- moved L3 156.2 mm to (227.6, 81.4), turned to 180 degrees
- moved L2 153.0 mm to (227.6, 76.8), turned to 180 degrees
- moved R4 143.1 mm to (223.9, 76.8), turned to 180 degrees
- moved R5 142.8 mm to (223.9, 81.4), turned to 180 degrees
- moved R133 140.9 mm to (162.2, 77.2), turned to 180 degrees
- moved R132 138.9 mm to (162.1, 85.1), turned to 180 degrees
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- renumbered C12 to C2, C3 to C216, C6 to C217, C4 to C218, C5 to C219, C8 to C220, C9 to C221, C10 to C222, C11 to C223, C13 to C3, C14 to C4, C15 to C5, C2 to C6, R3 to R1, R1 to R10, R2 to R11, R5 to R12, R4 to R2, R8 to R3, R9 to R4, R10 to R5, R11 to R8, R12 to R9, U3 to U2, U2 to U3
Connections:
- U5 pad G11: unconnected-(U5G-VCCBRAM-PadG11) -> +VCC_1V0
- U5 pad H10: unconnected-(U5G-VCCBRAM-PadH10) -> +VCC_1V0
- U5 pad N17: unconnected-(U5B-IO_L23P_T3_34-PadN17) -> /soc/soc-pl/DDR3_D12
- U5 pad N18: unconnected-(U5B-IO_L13P_T2_MRCC_34-PadN18) -> /soc/soc-pl/DDR3_ADDR14
- U5 pad N20: unconnected-(U5B-IO_L14P_T2_SRCC_34-PadN20) -> /soc/soc-pl/DDR3_BA1
- U5 pad P14: unconnected-(U5B-IO_L6P_T0_34-PadP14) -> /soc/soc-pl/DDR3_ADDR0
- U5 pad P15: unconnected-(U5B-IO_L24P_T3_34-PadP15) -> /soc/soc-pl/DDR3_D14
- U5 pad P16: unconnected-(U5B-IO_L24N_T3_34-PadP16) -> /soc/soc-pl/DDR3_D15
- U5 pad P18: unconnected-(U5B-IO_L23N_T3_34-PadP18) -> /soc/soc-pl/DDR3_D13
- U5 pad P19: unconnected-(U5B-IO_L13N_T2_MRCC_34-PadP19) -> /soc/soc-pl/DDR3_D5
- U5 pad P20: unconnected-(U5B-IO_L14N_T2_SRCC_34-PadP20) -> /soc/soc-pl/DDR3_BA2
- U5 pad R14: unconnected-(U5B-IO_L6N_T0_VREF_34-PadR14) -> /soc/soc-pl/DDR3_ADDR1
- U5 pad R16: unconnected-(U5B-IO_L19P_T3_34-PadR16) -> /soc/soc-pl/DDR3_CKE
- U5 pad R17: unconnected-(U5B-IO_L19N_T3_VREF_34-PadR17) -> /soc/soc-pl/DDR3_D7
- U5 pad R18: unconnected-(U5B-IO_L20N_T3_34-PadR18) -> /soc/soc-pl/DDR3_ODT0
- U5 pad R19: unconnected-(U5B-IO_0_34-PadR19) -> /soc/soc-pl/DDR3_D0
- U5 pad T10: unconnected-(U5B-IO_L1N_T0_34-PadT10) -> /soc/soc-pl/DDR3_D2
- U5 pad T11: unconnected-(U5B-IO_L1P_T0_34-PadT11) -> /soc/soc-pl/DDR3_D1
- U5 pad T12: unconnected-(U5B-IO_L2P_T0_34-PadT12) -> /soc/soc-pl/DDR3_D3
- U5 pad T14: unconnected-(U5B-IO_L5P_T0_34-PadT14) -> /soc/soc-pl/DDR3_DM0
- U5 pad T15: unconnected-(U5B-IO_L5N_T0_34-PadT15) -> /soc/soc-pl/DDR3_DM1
- U5 pad T16: unconnected-(U5B-IO_L9P_T1_DQS_34-PadT16) -> /soc/soc-pl/DDR3_ADDR6
- U5 pad T17: unconnected-(U5B-IO_L20P_T3_34-PadT17) -> /soc/soc-pl/DDR3_nCS
- U5 pad T20: unconnected-(U5B-IO_L15P_T2_DQS_34-PadT20) -> /soc/soc-pl/DDR3_D6
- U5 pad U12: unconnected-(U5B-IO_L2N_T0_34-PadU12) -> /soc/soc-pl/DDR3_D4
- U5 pad U13: unconnected-(U5B-IO_L3P_T0_DQS_PUDC_B_34-PadU13) -> /soc/soc-pl/DDR3_DQS0+
- U5 pad U14: unconnected-(U5B-IO_L11P_T1_SRCC_34-PadU14) -> /soc/soc-pl/DDR3_ADDR10
- U5 pad U15: unconnected-(U5B-IO_L11N_T1_SRCC_34-PadU15) -> /soc/soc-pl/DDR3_ADDR11
- U5 pad U17: unconnected-(U5B-IO_L9N_T1_DQS_34-PadU17) -> /soc/soc-pl/DDR3_ADDR7
- U5 pad U18: unconnected-(U5B-IO_L12P_T1_MRCC_34-PadU18) -> /soc/soc-pl/DDR3_ADDR12
- U5 pad U19: unconnected-(U5B-IO_L12N_T1_MRCC_34-PadU19) -> /soc/soc-pl/DDR3_ADDR13
- U5 pad U20: unconnected-(U5B-IO_L15N_T2_DQS_34-PadU20) -> /soc/soc-pl/DDR3_BA0
- U5 pad V12: unconnected-(U5B-IO_L4P_T0_34-PadV12) -> /soc/soc-pl/DDR3_DQS1+
- U5 pad V13: unconnected-(U5B-IO_L3N_T0_DQS_34-PadV13) -> /soc/soc-pl/DDR3_DQS0-
- U5 pad V15: unconnected-(U5B-IO_L10P_T1_34-PadV15) -> /soc/soc-pl/DDR3_ADDR8
- U5 pad V16: unconnected-(U5B-IO_L18P_T2_34-PadV16) -> /soc/soc-pl/DDR3_nWE
- U5 pad V17: unconnected-(U5B-IO_L21P_T3_DQS_34-PadV17) -> /soc/soc-pl/DDR3_D8
- U5 pad V18: unconnected-(U5B-IO_L21N_T3_DQS_34-PadV18) -> /soc/soc-pl/DDR3_D9
- U5 pad V20: unconnected-(U5B-IO_L16P_T2_34-PadV20) -> /soc/soc-pl/DDR3_CK+
- U5 pad W13: unconnected-(U5B-IO_L4N_T0_34-PadW13) -> /soc/soc-pl/DDR3_DQS1-
- U5 pad W14: unconnected-(U5B-IO_L8P_T1_34-PadW14) -> /soc/soc-pl/DDR3_ADDR4
- U5 pad W15: unconnected-(U5B-IO_L10N_T1_34-PadW15) -> /soc/soc-pl/DDR3_ADDR9
- U5 pad W16: unconnected-(U5B-IO_L18N_T2_34-PadW16) -> /soc/soc-pl/DDR3_nRST
- U5 pad W18: unconnected-(U5B-IO_L22P_T3_34-PadW18) -> /soc/soc-pl/DDR3_D10
- U5 pad W19: unconnected-(U5B-IO_L22N_T3_34-PadW19) -> /soc/soc-pl/DDR3_D11
- U5 pad W20: unconnected-(U5B-IO_L16N_T2_34-PadW20) -> /soc/soc-pl/DDR3_CK-
- U5 pad Y14: unconnected-(U5B-IO_L8N_T1_34-PadY14) -> /soc/soc-pl/DDR3_ADDR5
- U5 pad Y16: unconnected-(U5B-IO_L7P_T1_34-PadY16) -> /soc/soc-pl/DDR3_ADDR2
- U5 pad Y17: unconnected-(U5B-IO_L7N_T1_34-PadY17) -> /soc/soc-pl/DDR3_ADDR3
- U5 pad Y18: unconnected-(U5B-IO_L17P_T2_34-PadY18) -> /soc/soc-pl/DDR3_nRAS
- U5 pad Y19: unconnected-(U5B-IO_L17N_T2_34-PadY19) -> /soc/soc-pl/DDR3_nCAS
Routing:
- net +VCC_3V3: track 13.0 -> 72.0 mm, vias 23 -> 31
- net /soc/EMMC_D2: track 0.00 -> 40.2 mm, vias 0 -> 2
- net /soc/EMMC_D1: track 0.00 -> 35.2 mm, vias 0 -> 2
- net /eth-phy/ENET0_TXCLK: track 0.00 -> 29.1 mm, vias 0 -> 2
- net /soc/EMMC_D0: track 0.00 -> 29.0 mm, vias 0 -> 2
- net /eth-phy/ENET0_TXD1: track 0.00 -> 28.9 mm, vias 0 -> 2
- net /soc/FLSH_QSPI_IO0: track 0.00 -> 28.6 mm
- net /soc/EMMC_D3: track 0.00 -> 28.4 mm, vias 0 -> 2
- net +VCC_1V5: track 38.0 -> 64.9 mm
- net /eth-phy/ENET0_TXD3: track 0.00 -> 26.2 mm, vias 0 -> 2
- net +VCC_1V8: track 11.3 -> 35.3 mm
- net /soc/FLSH_QSPI_SCK: track 0.00 -> 21.1 mm
- net /soc/FLSH_QSPI_IO3: track 0.00 -> 19.7 mm
- net /soc/FLSH_QSPI_IO1: track 0.00 -> 18.9 mm
- net /eth-phy/ENET0_RXD3: track 0.00 -> 18.0 mm
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
Commit message: replaced pmic;
Parts:
- removed C12: CL21B475KPFNNNE, Capacitor_SMD:C_0805_2012Metric
- removed the C14 at (248.0, 71.3)
- removed the C213 at (224.9, 88.6)
- removed the C214 at (248.0, 69.3)
- removed the C3 at (241.8, 81.4)
- removed the L2 at (227.6, 76.8)
- removed the R5 at (223.9, 81.4)
- removed the R9 at (249.0, 81.4)
- added C1: CL21B475KPFNNNE, Capacitor_SMD:C_0805_2012Metric, F.Cu at (221.4, 43.0)
- added C218: CL21B475KPFNNNE, Capacitor_SMD:C_0805_2012Metric, F.Cu at (218.1, 21.6)
- added C219: CL21B475KPFNNNE, Capacitor_SMD:C_0805_2012Metric, F.Cu at (219.1, 27.4)
- added C220: CL21B106KQQNFNE, Capacitor_SMD:C_0805_2012Metric, F.Cu at (222.4, 21.5)
- added C221: CL21B475KPFNNNE, Capacitor_SMD:C_0805_2012Metric, F.Cu at (222.4, 19.4)
- added C6: CL21B106KQQNFNE, Capacitor_SMD:C_0805_2012Metric, F.Cu at (221.4, 45.0)
- added D5: 150060BS75000, LED_SMD:LED_0603_1608Metric, F.Cu at (266.6, 55.2)
- added L1: 74438357015, Inductors:WE-MAPI, F.Cu at (216.2, 41.1)
- added Q1: BSS138, Package_TO_SOT_SMD:SOT-23, F.Cu at (269.4, 55.3)
- added R11: RC0402FR-07100KL, Resistor_SMD:R_0402_1005Metric, F.Cu at (258.4, 45.1)
- added R12: RC0402FR-07100KL, Resistor_SMD:R_0402_1005Metric, F.Cu at (258.4, 47.1)
- added R135: RC0402FR-07100KL, Resistor_SMD:R_0402_1005Metric, F.Cu at (258.4, 49.1)
- added R136: RC0603FR-0710KL, Resistor_SMD:R_0603_1608Metric, F.Cu at (269.3, 52.9)
- added R146: RC0603FR-07220RL, Resistor_SMD:R_0603_1608Metric, F.Cu at (265.0, 55.1)
- added R3: RC0402FR-13470KL, Resistor_SMD:R_0402_1005Metric, F.Cu at (221.5, 40.3)
- added S4: 435441019830, Miscellaneous:435441019830, F.Cu at (268.2, 59.3)
- C10, C11, C8, C9: value CL31A106KBHNNNE -> CL21B475KPFNNNE; footprint Capacitor_SMD:C_1206_3216Metric_Pad1.33x1.80mm_HandSolder -> Capacitor_SMD:C_0805_2012Metric
- C13: value CL21B475KPFNNNE -> CL05B104KA5NNNC; footprint Capacitor_SMD:C_0805_2012Metric -> Capacitor_SMD:C_0402_1005Metric
- C15: value CL21B475KPFNNNE -> CL10B105KA8NNNC; footprint Capacitor_SMD:C_0805_2012Metric -> Capacitor_SMD:C_0603_1608Metric
- C194, C200: footprint Capacitor_SMD:C_0603_1608Metric_Pad1.08x0.95mm_HandSolder -> Capacitor_SMD:C_0603_1608Metric
- C195: footprint Capacitor_SMD:C_0402_1005Metric_Pad0.74x0.62mm_HandSolder -> Capacitor_SMD:C_0402_1005Metric
- C196, C197, C198, C199: footprint Capacitor_SMD:C_0805_2012Metric_Pad1.18x1.45mm_HandSolder -> Capacitor_SMD:C_0805_2012Metric
- C2, C4, C5: value CL31A106KBHNNNE -> CL21B106KQQNFNE; footprint Capacitor_SMD:C_1206_3216Metric -> Capacitor_SMD:C_0805_2012Metric
- C210, C211, R143, R144, U17, Y4: moved to B.Cu
- C212: value CL10B104KB8NNWC -> CL21B475KPFNNNE; footprint Capacitor_SMD:C_0603_1608Metric_Pad1.08x0.95mm_HandSolder -> Capacitor_SMD:C_0805_2012Metric
- C215: value CL10B104KB8NNWC -> CL21B106KQQNFNE; footprint Capacitor_SMD:C_0603_1608Metric_Pad1.08x0.95mm_HandSolder -> Capacitor_SMD:C_0805_2012Metric
- L3, L4, L5: value DFE322512F-R47M=P2 -> 74438357015; footprint Inductors:IND_1210 -> Inductors:WE-MAPI
- R100, R101, R102, R103, R104, R105, R106, R107, R108, R109, R110, R111, R112, R113, R114, R115, R116, R117, R118, R131, R134, R22, R23, R27, R28, R29, R30, R95, R96, R97, R98, R99: footprint Resistor_SMD:R_0402_1005Metric_Pad0.72x0.64mm_HandSolder -> Resistor_SMD:R_0402_1005Metric
- R127, R128, R129, R130, R132, R133, R138, R141, R145: footprint Resistor_SMD:R_0603_1608Metric_Pad0.98x0.95mm_HandSolder -> Resistor_SMD:R_0603_1608Metric
- R4: value RC0603JR-070RL -> RC0402FR-07100KL; footprint Resistor_SMD:R_0603_1608Metric -> Resistor_SMD:R_0402_1005Metric
- R8: value RC0603JR-070RL -> RC0603FR-0720KL; footprint Resistor_SMD:R_0603_1608Metric -> Resistor_SMD:R_0201_0603Metric
- U2: value LP8758A1E0YFFR -> TPS65218D0RSLT; footprint ICs:R-XBGA-N35 -> ICs:RSL0048G
- moved R1 171.5 mm to (247.5, 45.3)
- moved R2 171.5 mm to (247.5, 47.8)
- moved C215 75.2 mm to (218.1, 19.7)
- moved C2 62.0 mm to (226.5, 19.6), turned to 0 degrees
- moved L5 61.1 mm to (222.3, 24.8), turned to 180 degrees
- moved C11 60.1 mm to (213.9, 34.8)
- moved L4 59.5 mm to (214.3, 26.0), turned to -90 degrees
- moved C15 57.4 mm to (228.3, 32.8), turned to 0 degrees
- moved U17 56.6 mm to (163.8, 95.4), turned to 90 degrees
- moved L3 56.6 mm to (226.8, 24.8), turned to 0 degrees
- moved R144 54.9 mm to (168.8, 93.1), turned to 0 degrees
- moved C211 54.0 mm to (171.1, 92.3), turned to 90 degrees
- moved R143 54.0 mm to (168.8, 94.6), turned to 0 degrees
- moved C210 52.5 mm to (171.1, 95.4), turned to -90 degrees
- moved C8 52.2 mm to (226.5, 21.6)
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- renumbered C6 to C14, C216 to C213, C217 to C214, C218 to C216, C219 to C217, C220 to C222, C221 to C223, C222 to C224, C223 to C225, C1 to C3, L1 to L2, R11 to R10, R12 to R147, R3 to R5, R10 to R9
Connections:
- C10 pad 1: +VCC_1V2 -> +VIN_5V0
- C11 pad 1: +VCC_1V8 -> +VIN_5V0
- C13 pad 1: +PS_VCC_1V5 -> Net-(U2-PFI)
- C14 pad 1: +VCC_3V3 -> +LDO_3V3
- C15 pad 1: +VCC_1V8 -> Net-(U2-INT_LDO)
- C2 pad 1: +VIN_5V0 -> +VCC_1V5
- C212 pad 1: +VCC_1V0 -> +VIN_5V0
- C215 pad 1: +VCC_1V8 -> +VCC_1V0
- C4 pad 1: GND -> +VCC_1V8
- C4 pad 2: +VIN_5V0 -> GND
- C46 pad 1: +VCC_1V5 -> +VCC_DDR_1V5
- C47 pad 1: +VCC_1V5 -> +VCC_DDR_1V5
- C49 pad 1: +VCC_1V5 -> +VCC_DDR_1V5
- C5 pad 1: GND -> +VCC_DDR_1V5
- C5 pad 2: +VIN_5V0 -> GND
- C51 pad 1: +VCC_1V5 -> +VCC_DDR_1V5
- C57 pad 1: +VCC_1V5 -> +VCC_DDR_1V5
- C63 pad 1: +VCC_1V5 -> +VCC_DDR_1V5
- C8 pad 1: +VCC_1V0 -> +VCC_1V5
- C9 pad 1: +PS_VCC_1V5 -> +VIN_5V0
- L2 pad 2: +VCC_3V3 -> +LDO_3V3
- L3 pad 1: Net-(L3-Pad1) -> +VCC_1V5
- L3 pad 2: Net-(U2-FB_B1) -> Net-(U2-L3)
- L4 pad 1: Net-(L4-Pad1) -> +VCC_1V0
- L4 pad 2: Net-(U2-FB_B2) -> Net-(U2-L1)
- L5 pad 1: Net-(L5-Pad1) -> +VCC_1V2
- L5 pad 2: Net-(U2-FB_B3) -> Net-(U2-L2)
- R1 pad 1: Net-(U2-~{INT}) -> +LDO_3V3
- R1 pad 2: +VCC_3V3 -> /mcu/ST_I2C1_SDA
- R2 pad 1: Net-(U2-~{RST}) -> +LDO_3V3
- R2 pad 2: +VCC_3V3 -> /mcu/ST_I2C1_SCL
- R4 pad 1: Net-(U2-FB_B0) -> Net-(U2-PFI)
- R4 pad 2: +VCC_1V0 -> GND
- R5 pad 2: +VCC_3V3 -> +LDO_3V3
- R8 pad 1: Net-(U2-FB_B2) -> Net-(U2-DC34_SEL)
- R8 pad 2: +VCC_1V2 -> GND
- U1 pad 3: +VCC_3V3 -> +LDO_3V3
- U1 pad 4: +VCC_3V3 -> +LDO_3V3
- U5 pad A3: +VCC_1V5 -> +VCC_DDR_1V5
- U5 pad D2: +VCC_1V5 -> +VCC_DDR_1V5
- U5 pad E5: +VCC_1V5 -> +VCC_DDR_1V5
- U5 pad G1: +VCC_1V5 -> +VCC_DDR_1V5
- U5 pad H4: +VCC_1V5 -> +VCC_DDR_1V5
- U5 pad L3: +VCC_1V5 -> +VCC_DDR_1V5
- U5 pad P2: +VCC_1V5 -> +VCC_DDR_1V5
- U5 pad R5: +VCC_1V5 -> +VCC_DDR_1V5
- U5 pad U1: +VCC_1V5 -> +VCC_DDR_1V5
- U5 pad V4: +VCC_1V5 -> +VCC_DDR_1V5
Routing:
- net /soc/soc-ps/USB0_CLK: track 2.54 -> 42.8 mm
- net /eth-phy/ENET0_TXD2: track 0.57 -> 34.5 mm, vias 1 -> 2
- net /soc/soc-ps/USB0_DATA7: track 7.51 -> 33.4 mm
- net /soc/soc-ps/USB0_DATA0: track 12.0 -> 34.3 mm
- net /eth-phy/ENET0_RXD0: track 0.57 -> 21.5 mm, vias 1 -> 2
- net /eth-phy/ENET0_RXCTL: track 0.57 -> 18.7 mm, vias 1 -> 2
- net /soc/soc-ps/USB0_DATA4: track 10.5 -> 27.2 mm
- net +VIN_5V0: track 1.60 -> 15.5 mm
- net +VCC_1V0: track 32.0 -> 45.0 mm
- net /soc/soc-ps/USB0_DATA2: track 18.8 -> 31.4 mm
- net /soc/soc-ps/USB0_DATA5: track 20.8 -> 30.8 mm
- net +PS_VTT_0V75: track 7.56 -> 17.4 mm, vias 2 -> 16
- net /soc/soc-ps/USB0_DATA1: track 15.0 -> 24.6 mm
- net /soc/soc-ps/USB0_DATA6: track 17.3 -> 26.8 mm
- net Net-(U2-L1): track 0.00 -> 9.08 mm
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- removed copper zone on F.Cu, net +VIN_5V0
- removed copper zone on F.Cu, net GND
- removed copper zone on F.Cu, net Net-(L2-Pad1)
- removed copper zone on F.Cu, net Net-(L3-Pad1)
- removed copper zone on F.Cu, net Net-(L4-Pad1)
- removed copper zone on F.Cu, net Net-(L5-Pad1)
