File: Hardware/Design Files/rfsom-01/rfsom-01.kicad_pcb (KiCad board)
At the start: 10 copper layers, 102.2 x 100 mm, 432 parts, among them J1 TC2050, J10 SEAM-40-02.0-L-04-2-A-K-TR, J2 2216100001, J3 SEAM-40-02.0-L-04-2-A-K-TR, J9 DM3CS-SF, Q1 BSS138, U1 TPS62086RLT, U10 STM32L432KCUx, U11 AS4C256M16D3C-12BCN, U12 TPS51200DRCR, U13 S25FL128SAGNFI003, U14 MX52LM04A11XSI, U16 93LC56BT-I/OT, U17 USB3320C-EZK, U2 TPS65218D0RSLT, U3 TPS51200DRCR, U4 FT232HQ-REEL, U5 XC7Z010-1CLG400C, U6 KSZ9131RNXI-TR, U7 TXS02612RTWR, U8 AS4C256M16D3C-12BCN, U9 AS4C256M16D3C-12BCN, Y1 ECS-2033-500-BN, Y2 ABM10-166-12.000MHZ-T3, Y3 ECS-2033-250-BN, Y4 ECS-240-12-37B-CKY-TR

Commit message: aorus refresh;
Parts:
- C1, C10, C11, C13, C15, C2, C212, C215, C218, C219, C220, C221, C4, C5, C56, C6, C71, C74, C8, C9, L1, L3, L4, L5, R3, R4, R8, U2: moved to B.Cu
- U17: footprint Package_DFN_QFN:QFN-32-1EP_5x5mm_P0.5mm_EP3.1x3.1mm -> ICs:QFN-32-1EP_5x5mm_P0.5mm
- moved C215 102.1 mm to (182.4, 115.3), turned to 0 degrees
- moved C218 102.0 mm to (182.4, 117.2), turned to 0 degrees
- moved L4 97.2 mm to (178.4, 116.3), turned to 180 degrees
- moved C221 95.8 mm to (186.5, 108.2), turned to -90 degrees
- moved C220 94.7 mm to (184.4, 108.2), turned to -90 degrees
- moved C212 94.3 mm to (175.2, 116.7), turned to -90 degrees
- moved C2 93.6 mm to (186.3, 104.1), turned to 90 degrees
- moved C4 93.3 mm to (173.1, 116.7), turned to -90 degrees
- moved L5 93.1 mm to (181.1, 108.3), turned to -90 degrees
- moved C219 92.9 mm to (176.4, 109.9), turned to -90 degrees
- moved C8 92.7 mm to (184.3, 104.1), turned to 90 degrees
- moved C11 92.4 mm to (171.1, 116.7), turned to -90 degrees
- moved C9 91.6 mm to (169.1, 116.7), turned to -90 degrees
- moved L3 91.3 mm to (181.1, 103.8), turned to 90 degrees
- moved U2 89.6 mm to (171.3, 108.3), turned to 90 degrees
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Connections:
- C46 pad 1: +VCC_DDR_1V5 -> +VCC_1V5
- C47 pad 1: +VCC_DDR_1V5 -> +VCC_1V5
- C49 pad 1: +VCC_DDR_1V5 -> +VCC_1V5
- C51 pad 1: +VCC_DDR_1V5 -> +VCC_1V5
- C57 pad 1: +VCC_DDR_1V5 -> +VCC_1V5
- C63 pad 1: +VCC_DDR_1V5 -> +VCC_1V5
- U5 pad A3: +VCC_DDR_1V5 -> +VCC_1V5
- U5 pad D2: +VCC_DDR_1V5 -> +VCC_1V5
- U5 pad E5: +VCC_DDR_1V5 -> +VCC_1V5
- U5 pad G1: +VCC_DDR_1V5 -> +VCC_1V5
- U5 pad H4: +VCC_DDR_1V5 -> +VCC_1V5
- U5 pad L3: +VCC_DDR_1V5 -> +VCC_1V5
- U5 pad P2: +VCC_DDR_1V5 -> +VCC_1V5
- U5 pad R5: +VCC_DDR_1V5 -> +VCC_1V5
- U5 pad U1: +VCC_DDR_1V5 -> +VCC_1V5
- U5 pad V4: +VCC_DDR_1V5 -> +VCC_1V5
Routing:
- net +VCC_3V3: track 77.7 -> 23.4 mm, vias 31 -> 33
- net /soc/soc-ram/DDR3_ADDR11: track 22.3 -> 68.7 mm
- net /soc/soc-ram/DDR3_ADDR14: track 22.6 -> 65.0 mm
- net +VCC_1V5: track 72.7 -> 38.0 mm
- net /soc/soc-ram/DDR3_ADDR12: track 25.7 -> 57.3 mm
- net /soc/soc-ps/USB0_DATA7: track 33.4 -> 6.55 mm
- net /soc/soc-ram/DDR3_ADDR8: track 20.3 -> 46.6 mm
- net +VCC_1V8: track 40.2 -> 14.0 mm, vias 16 -> 17
- net /soc/soc-ram/DDR3_ADDR1: track 23.6 -> 49.7 mm
- net +VCC_1V0: track 45.0 -> 19.2 mm, vias 17 -> 18
- net /soc/soc-ram/DDR3_ADDR6: track 19.6 -> 44.6 mm
- net /soc/soc-ram/DDR3_ADDR10: track 13.6 -> 38.1 mm
- net /soc/soc-ram/DDR3_ADDR13: track 22.9 -> 46.7 mm
- net /soc/soc-ram/DDR3_ADDR2: track 26.5 -> 49.9 mm
- net /soc/soc-ram/DDR3_ADDR4: track 21.5 -> 44.4 mm
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- added copper zone on In2.Cu, net +ETH_AVDDH
- added copper zone on In2.Cu, net +ETH_AVDDL
- added copper zone on In2.Cu, net +ETH_DVDDH
- added copper zone on In2.Cu, net +ETH_DVDDL
- added copper zone on In2.Cu, net +VCC_1V0
- added copper zone on B.Cu, net +VCC_1V2
- added copper zone on In8.Cu, net +VCC_1V2
- added copper zone on B.Cu, net +VCC_1V5
- added copper zone on In2.Cu, net +VCC_1V5
- added copper zone on In8.Cu, net +VCC_1V8
- added copper zone on In2.Cu, net +VCC_3V3
- added copper zone on B.Cu, net +VIN_5V0
- added copper zone on B.Cu, net Net-(U2-L2)
- added copper zone on B.Cu, net Net-(U2-L3)
