File: Hardware/Design Files/rfsom-01/rfsom-01.kicad_pcb (KiCad board)
At the start: 10 copper layers, 102.2 x 100 mm, 432 parts, among them J1 TC2050, J10 SEAM-40-02.0-L-04-2-A-K-TR, J2 2216100001, J3 SEAM-40-02.0-L-04-2-A-K-TR, J9 DM3CS-SF, Q1 BSS138, U1 TPS62086RLT, U10 STM32L432KCUx, U11 AS4C256M16D3C-12BCN, U12 TPS51200DRCR, U13 S25FL128SAGNFI003, U14 MX52LM04A11XSI, U16 93LC56BT-I/OT, U17 USB3320C-EZK, U2 TPS65218D0RSLT, U3 TPS51200DRCR, U4 FT232HQ-REEL, U5 XC7Z010-1CLG400C, U6 KSZ9131RNXI-TR, U7 TXS02612RTWR, U8 AS4C256M16D3C-12BCN, U9 AS4C256M16D3C-12BCN, Y1 ECS-2033-500-BN, Y2 ABM10-166-12.000MHZ-T3, Y3 ECS-2033-250-BN, Y4 ECS-240-12-37B-CKY-TR

Commit message: restructured project;
Routing:
- net /soc/soc-pl/DDR3_ADDR6: vias 1 -> 0
- net +VCC_3V3: vias 33 -> 34
