File: Hardware/Design Files/rfsom-01/mcu.kicad_sch (KiCad schematic)
At the start: 10 parts, among them U10 STM32L432KCUx

Commit message: aorus refresh;
Parts:
- removed C76: CL21B475KPFNNNE, Capacitor_SMD:C_0805_2012Metric, symbol Capacitors:CL21B475KPFNNNE
- removed C77, C78: CL10B105KA8NNNC, Capacitor_SMD:C_0603_1608Metric, symbol Capacitors:CL10B105KA8NNNC
- removed C79, C81: CL05B104KA5NNNC, Capacitor_SMD:C_0402_1005Metric, symbol Capacitors:CL05B104KA5NNNC
- removed C80: CL05B103KB5NNNC, Capacitor_SMD:C_0402_1005Metric, symbol Capacitors:CL05B103KB5NNNC
- removed R24: RC0402FR-07100KL, Resistor_SMD:R_0402_1005Metric, symbol Resistors:RC0402FR-07100KL
- removed R25, R26: RC0603FR-0710KL, Resistor_SMD:R_0603_1608Metric, symbol Resistors:RC0603FR-0710KL
- removed U10: STM32L432KCUx, Package_DFN_QFN:QFN-32-1EP_5x5mm_P0.5mm_EP3.45x3.45mm, symbol MCU_ST_STM32L4:STM32L432KCUx
Other:
- note removed: "VDD"
- note removed: "VDDA"
