File: Hardware/Design Files/rfsom-01/power.kicad_sch (KiCad schematic)
At the start: 53 parts, among them Q1 BSS138, U1 TPS62086RLT, U2 TPS65218D0RSLT, U3 TPS51200DRCR

Commit message: aorus refresh;
Parts:
- removed C1, C10, C11, C12, C212, C213, C218, C219, C221, C8, C9: CL21B475KPFNNNE, Capacitor_SMD:C_0805_2012Metric, symbol Capacitors:CL21B475KPFNNNE
- removed C13, C222: CL05B104KA5NNNC, Capacitor_SMD:C_0402_1005Metric, symbol Capacitors:CL05B104KA5NNNC
- removed C14: GRM188R60G106ME47, Capacitor_SMD:C_0603_1608Metric, symbol Capacitors:GRM188R60G106ME47
- removed C15: CL10B105KA8NNNC, Capacitor_SMD:C_0603_1608Metric, symbol Capacitors:CL10B105KA8NNNC
- removed C2, C215, C216, C217, C220, C223, C224, C225, C4, C5, C6: CL21B106KQQNFNE, Capacitor_SMD:C_0805_2012Metric, symbol Capacitors:CL21B106KQQNFNE
- removed C214: CL05B102KB5NNNC, Capacitor_SMD:C_0402_1005Metric, symbol Capacitors:CL05B102KB5NNNC
- removed C3: CL21B475KAFNNNE, Capacitor_SMD:C_0805_2012Metric, symbol Capacitors:CL21B475KAFNNNE
- removed D5: 150060BS75000, LED_SMD:LED_0603_1608Metric, symbol Diodes:150060BS75000
- removed L1, L3, L4, L5: 74438357015, Inductors:WE-MAPI, symbol Inductors:74438357015
- removed L2: DFE322512F-R47M=P2, Inductors:IND_1210, symbol Inductors:DFE322512F-R47M=P2
- removed Q1: BSS138, Package_TO_SOT_SMD:SOT-23, symbol Transistor_FET:BSS138
- removed R1, R10, R136, R2, R9: RC0603FR-0710KL, Resistor_SMD:R_0603_1608Metric, symbol Resistors:RC0603FR-0710KL
- removed R11, R12, R135, R147, R4, R5: RC0402FR-07100KL, Resistor_SMD:R_0402_1005Metric, symbol Resistors:RC0402FR-07100KL
- removed R146: RC0603FR-07220RL, Resistor_SMD:R_0603_1608Metric, symbol Resistors:RC0603FR-07220RL
- removed R3: RC0402FR-13470KL, Resistor_SMD:R_0402_1005Metric, symbol Resistors:RC0402FR-13470KL
- removed R8: RC0603FR-0720KL, Resistor_SMD:R_0201_0603Metric, symbol Resistors:RC0603FR-0720KL
- removed S4: 435441019830, Miscellaneous:435441019830, symbol Miscellaneous:435441019830
- removed U1: TPS62086RLT, ICs:RLT0007A, symbol ICs:TPS62086RLT
- removed U2: TPS65218D0RSLT, ICs:RSL0048G, symbol ICs:TPS65218D0RSLT
- removed U3: TPS51200DRCR, Package_SON:VSON-10-1EP_3x3mm_P0.5mm_EP1.65x2.4mm, symbol ICs:TPS51200DRCR
Connections:
- no-connect marks 4 -> 0
Other:
- note removed: "0.3A"
- note removed: "0.4A"
- note removed: "0.9A"
- note removed: "1.0A"
- note removed: "1.8A"
- note removed: "3A OUT"
- note removed: "PFI SET TO 4.56V THRESHOLD."
- note removed: "V CCPINT -> VCCPAUX, VCCPLL -> VCCO_MIO0, VCCO_MIO1, VCCO_DDR 1 (2.5A) -> 1.8V (1.5A), 1.8V (100mA) -> 3.3V (2.0A), 1.5 (2.5A)"
