File: Hardware/Design Files/rfsom-01/[01] - top.kicad_sch (KiCad schematic)
At the start: 3 parts, among them J1 TC2050

Commit message: restructured project;
Other:
- sheet mcu: file mcu.kicad_sch -> [03] - mcu.kicad_sch
- sheet power: file power.kicad_sch -> [02] - power.kicad_sch
Changed lines of the file:
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@@
+				)
+			)
+			(project "rfsom-01"
+				(path "/abe8d823-e11a-4177-8ce6-4f279cf45b05/8f56564b-be87-47cb-af1d-0a8f839d3522"
+					(reference "H2")
+					(unit 1)
 				)
 			)
@@
 		(dnp no)
 		(fields_autoplaced yes)
-		(property "Reference" "#PWR084"
+		(property "Reference" "#PWR014"
 			(at 53.34 49.53 0)
 			(hide yes)
@@
 				(path "/5dade83d-850c-4336-8f49-e0e8e6ebca37"
 					(reference "#PWR084")
+					(unit 1)
+				)
+			)
+			(project "rfsom-01"
+				(path "/abe8d823-e11a-4177-8ce6-4f279cf45b05/8f56564b-be87-47cb-af1d-0a8f839d3522"
+					(reference "#PWR014")
 					(unit 1)
 				)
@@
 			(project "[01] - rfsom-01"
 				(path "/5dade83d-850c-4336-8f49-e0e8e6ebca37"
+					(reference "J1")
+					(unit 1)
+				)
+			)
+			(project "rfsom-01"
+				(path "/abe8d823-e11a-4177-8ce6-4f279cf45b05/8f56564b-be87-47cb-af1d-0a8f839d3522"
 					(reference "J1")
 					(unit 1)
@@
 				)
 			)
+			(project "rfsom-01"
+				(path "/abe8d823-e11a-4177-8ce6-4f279cf45b05/8f56564b-be87-47cb-af1d-0a8f839d3522"
+					(reference "H1")
+					(unit 1)
+				)
+			)
 		)
 	)
@@
 		(dnp no)
 		(fields_autoplaced yes)
-		(property "Reference" "#PWR098"
+		(property "Reference" "#PWR06"
 			(at 33.02 26.67 0)
 			(hide yes)
@@
 				(path "/5dade83d-850c-4336-8f49-e0e8e6ebca37"
 					(reference "#PWR098")
+					(unit 1)
+				)
+			)
+			(project "rfsom-01"
+				(path "/abe8d823-e11a-4177-8ce6-4f279cf45b05/8f56564b-be87-47cb-af1d-0a8f839d3522"
+					(reference "#PWR06")
 					(unit 1)
 				)
@@
 		(dnp no)
 		(fields_autoplaced yes)
-		(property "Reference" "#PWR0208"
+		(property "Reference" "#PWR04"
 			(at 26.67 138.43 0)
 			(hide yes)
@@
 				(path "/5dade83d-850c-4336-8f49-e0e8e6ebca37"
 					(reference "#PWR0208")
+					(unit 1)
+				)
+			)
+			(project "rfsom-01"
+				(path "/abe8d823-e11a-4177-8ce6-4f279cf45b05/8f56564b-be87-47cb-af1d-0a8f839d3522"
+					(reference "#PWR04")
 					(unit 1)
 				)
@@
 		(dnp no)
 		(fields_autoplaced yes)
-		(property "Reference" "#PWR0207"
+		(property "Reference" "#PWR03"
 			(at 20.32 132.08 0)
 			(hide yes)
@@
 				(path "/5dade83d-850c-4336-8f49-e0e8e6ebca37"
 					(reference "#PWR0207")
+					(unit 1)
+				)
+			)
+			(project "rfsom-01"
+				(path "/abe8d823-e11a-4177-8ce6-4f279cf45b05/8f56564b-be87-47cb-af1d-0a8f839d3522"
+					(reference "#PWR03")
 					(unit 1)
 				)
@@
 				)
 			)
+			(project ""
+				(path "/8f56564b-be87-47cb-af1d-0a8f839d3522"
+					(page "#")
+				)
+			)
+			(project "rfsom-01"
+				(path "/abe8d823-e11a-4177-8ce6-4f279cf45b05/8f56564b-be87-47cb-af1d-0a8f839d3522"
+					(page "17")
+				)
+			)
 		)
 	)
@@
 				)
 			)
+			(project ""
+				(path "/8f56564b-be87-47cb-af1d-0a8f839d3522"
+					(page "#")
+				)
+			)
+			(project "rfsom-01"
+				(path "/abe8d823-e11a-4177-8ce6-4f279cf45b05/8f56564b-be87-47cb-af1d-0a8f839d3522"
+					(page "3")
+				)
+			)
 		)
 	)
@@
 			)
 		)
-		(property "Sheetfile" "power.kicad_sch"
+		(property "Sheetfile" "[02] - power.kicad_sch"
 			(at 158.75 43.7646 0)
 			(show_name no)
@@
 				(path "/5dade83d-850c-4336-8f49-e0e8e6ebca37"
 					(page "2")
+				)
+			)
+			(project ""
+				(path "/8f56564b-be87-47cb-af1d-0a8f839d3522"
+					(page "#")
+				)
+			)
+			(project "rfsom-01"
+				(path "/abe8d823-e11a-4177-8ce6-4f279cf45b05/8f56564b-be87-47cb-af1d-0a8f839d3522"
+					(page "15")
 				)
 			)
@@
 				)
 			)
+			(project ""
+				(path "/8f56564b-be87-47cb-af1d-0a8f839d3522"
+					(page "#")
+				)
+			)
+			(project "rfsom-01"
+				(path "/abe8d823-e11a-4177-8ce6-4f279cf45b05/8f56564b-be87-47cb-af1d-0a8f839d3522"
+					(page "16")
+				)
+			)
 		)
 	)
@@
 			)
 		)
-		(property "Sheetfile" "mcu.kicad_sch"
+		(property "Sheetfile" "[03] - mcu.kicad_sch"
 			(at 109.22 43.7646 0)
 			(show_name no)
@@
 				(path "/5dade83d-850c-4336-8f49-e0e8e6ebca37"
 					(page "3")
+				)
+			)
+			(project ""
+				(path "/8f56564b-be87-47cb-af1d-0a8f839d3522"
+					(page "#")
+				)
+			)
+			(project "rfsom-01"
+				(path "/abe8d823-e11a-4177-8ce6-4f279cf45b05/8f56564b-be87-47cb-af1d-0a8f839d3522"
+					(page "13")
 				)
 			)
@@
 				)
 			)
+			(project ""
+				(path "/8f56564b-be87-47cb-af1d-0a8f839d3522"
+					(page "#")
+				)
+			)
+			(project "rfsom-01"
+				(path "/abe8d823-e11a-4177-8ce6-4f279cf45b05/8f56564b-be87-47cb-af1d-0a8f839d3522"
+					(page "14")
+				)
+			)
 		)
 	)
-	(sheet_instances
-		(path "/"
-			(page "1")
-		)
-	)
-	(embedded_fonts no)
 )
