File: Hardware/Design Files/rfsom-01/[02] - power.kicad_sch (KiCad schematic)
At the start: 52 parts, among them Q1 BSS138, U1 TPS62086RLT, U2 TPS65218D0RSLT, U3 TPS51200DRCR

Commit message: restructured project;
Parts:
- renumbered C1 to C198, C2 to C199, C3 to C200, C4 to C201, C5 to C202, C6 to C203, C8 to C204, C9 to C205, C10 to C206, C11 to C207, C13 to C208, C14 to C209, C15 to C210, C212 to C211, C213 to C212, C214 to C213, C215 to C214, C216 to C215, C217 to C216, C218 to C217, C219 to C218, C220 to C219, C221 to C220, C222 to C221, C223 to C222, C224 to C223, C225 to C224, R1 to R134, R2 to R135, R3 to R136, R4 to R137, R5 to R138, R8 to R139, R9 to R140, R10 to R141, R11 to R142, R12 to R143, R135 to R144, R136 to R145, U1 to U14, U2 to U15, U3 to U16
