File: Hardware/Design Files/rfsom-01/[03] - mcu.kicad_sch (KiCad schematic)
At the start: 10 parts, among them U10 STM32L432KCUx

Commit message: restructured project;
Parts:
- renumbered C76 to C169, C77 to C170, C78 to C171, C79 to C172, C80 to C173, C81 to C174, R24 to R112, R25 to R113, R26 to R114, U10 to U12
