File: Hardware/Design Files/rfsom-01/[05] - soc-power.kicad_sch (KiCad schematic)
At the start: 54 parts, among them U5 XC7Z010-1CLG400C

Commit message: restructured project;
Parts:
- renumbered C46 to C25, C47 to C26, C48 to C27, C49 to C28, C50 to C29, C51 to C30, C52 to C31, C53 to C32, C54 to C33, C55 to C34, C56 to C35, C57 to C36, C58 to C37, C59 to C38, C60 to C39, C61 to C40, C62 to C41, C63 to C42, C64 to C43, C65 to C44, C66 to C45, C67 to C46, C68 to C47, C163 to C48, C69 to C49, C70 to C50, C71 to C51, C72 to C52, C73 to C53, C74 to C54, C75 to C55, C82 to C56, C83 to C57, C84 to C58, C85 to C59, C86 to C60, C87 to C61, C88 to C62, C89 to C63, C90 to C64, C91 to C65, C92 to C66, C93 to C67, C94 to C68, C95 to C69, C96 to C70, C97 to C71, C98 to C72, C99 to C73, C100 to C74, C101 to C75, C102 to C76, C103 to C77, U5 to U6
