File: Hardware/Design Files/rfsom-01/[06] - soc-ps.kicad_sch (KiCad schematic)
At the start: 42 parts, among them U5 XC7Z010-1CLG400C, Y1 ECS-2033-500-BN

Commit message: restructured project;
Parts:
- renumbered C104 to C159, C106 to C160, C107 to C161, C108 to C162, C7 to C163, FB10 to FB5, FB11 to FB6, R61 to R100, R62 to R101, R63 to R102, R64 to R103, R65 to R104, R66 to R105, R67 to R106, R42 to R83, R43 to R84, R45 to R85, R46 to R86, R47 to R87, R48 to R88, R50 to R89, R51 to R90, R49 to R91, R53 to R92, R54 to R93, R55 to R94, R56 to R95, R57 to R96, R58 to R97, R59 to R98, R60 to R99, U5 to U6, Y1 to Y2
