File: Hardware/Design Files/rfsom-01/[07] - soc-ddr.kicad_sch (KiCad schematic)
At the start: 64 parts, among them U5 XC7Z010-1CLG400C

Commit message: restructured project;
Parts:
- renumbered C111 to C78, C112 to C79, C113 to C80, C114 to C81, C115 to C82, C116 to C83, C117 to C84, C118 to C85, C119 to C86, C120 to C87, R68 to R24, R69 to R25, R70 to R26, R71 to R27, R72 to R28, R73 to R29, R74 to R30, R75 to R31, R76 to R32, R77 to R33, R78 to R34, R79 to R35, R80 to R36, R81 to R37, R82 to R38, R83 to R39, R84 to R40, R85 to R41, R86 to R42, R87 to R43, R88 to R44, R89 to R45, R90 to R46, R91 to R47, R92 to R48, R93 to R49, R95 to R50, R96 to R51, R97 to R52, R98 to R53, R99 to R54, R100 to R55, R101 to R56, R102 to R57, R103 to R58, R104 to R59, R105 to R60, R106 to R61, R107 to R62, R108 to R63, R109 to R64, R94 to R65, R110 to R66, R111 to R67, R112 to R68, R113 to R69, R114 to R70, R115 to R71, R116 to R72, R117 to R73, R118 to R74, R119 to R75, R120 to R76, U5 to U6
