File: Hardware/Design Files/rfsom-01/[08] - ram.kicad_sch (KiCad schematic)
At the start: 23 parts, among them U11 AS4C256M16D3C-12BCN

Commit message: restructured project;
Parts:
- renumbered C148 to C100, C149 to C101, C150 to C102, C155 to C103, C156 to C104, C157 to C105, C158 to C106, C161 to C107, C162 to C108, C126 to C88, C127 to C89, C128 to C90, C129 to C91, C130 to C92, C136 to C93, C137 to C94, C138 to C95, C139 to C96, C140 to C97, C146 to C98, C147 to C99, R122 to R77, U11 to U7
