File: Hardware/Design Files/rfsom-01/[09] - soc-pl.kicad_sch (KiCad schematic)
At the start: 1 part, among them U5 XC7Z010-1CLG400C

Commit message: restructured project;
Parts:
- renumbered U5 to U6
Changed lines of the file:
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@@
 		(dnp no)
 		(fields_autoplaced yes)
-		(property "Reference" "U5"
+		(property "Reference" "U6"
 			(at 40.64 22.86 0)
 			(show_name no)
@@
 				(path "/5dade83d-850c-4336-8f49-e0e8e6ebca37/5824b29f-0639-4332-9093-651d63d89232/dcd4ebf5-9bf5-4a13-8e67-04058a43970d"
 					(reference "U5")
+					(unit 2)
+				)
+			)
+			(project "rfsom-01"
+				(path "/abe8d823-e11a-4177-8ce6-4f279cf45b05/8f56564b-be87-47cb-af1d-0a8f839d3522/5824b29f-0639-4332-9093-651d63d89232/dcd4ebf5-9bf5-4a13-8e67-04058a43970d"
+					(reference "U6")
 					(unit 2)
 				)
@@
 		(dnp no)
 		(fields_autoplaced yes)
-		(property "Reference" "U5"
+		(property "Reference" "U6"
 			(at 142.24 22.86 0)
 			(show_name no)
@@
 				(path "/5dade83d-850c-4336-8f49-e0e8e6ebca37/5824b29f-0639-4332-9093-651d63d89232/dcd4ebf5-9bf5-4a13-8e67-04058a43970d"
 					(reference "U5")
+					(unit 3)
+				)
+			)
+			(project "rfsom-01"
+				(path "/abe8d823-e11a-4177-8ce6-4f279cf45b05/8f56564b-be87-47cb-af1d-0a8f839d3522/5824b29f-0639-4332-9093-651d63d89232/dcd4ebf5-9bf5-4a13-8e67-04058a43970d"
+					(reference "U6")
 					(unit 3)
 				)
@@
 				)
 			)
+			(project ""
+				(path "/8f56564b-be87-47cb-af1d-0a8f839d3522/5824b29f-0639-4332-9093-651d63d89232/dcd4ebf5-9bf5-4a13-8e67-04058a43970d"
+					(page "#")
+				)
+			)
+			(project "rfsom-01"
+				(path "/abe8d823-e11a-4177-8ce6-4f279cf45b05/8f56564b-be87-47cb-af1d-0a8f839d3522/5824b29f-0639-4332-9093-651d63d89232/dcd4ebf5-9bf5-4a13-8e67-04058a43970d"
+					(page "10")
+				)
+			)
