File: Hardware/Design Files/rfsom-01/[11] - storage.kicad_sch (KiCad schematic)
At the start: 18 parts, among them J9 DM3CS-SF, U13 S25FL128SAGNFI003, U14 MX52LM04A11XSI

Commit message: restructured project;
Parts:
- renumbered C194 to C19, C195 to C20, C196 to C21, C197 to C22, C198 to C23, C110 to C24, J9 to J6, R127 to R15, R128 to R16, R129 to R17, R130 to R18, R131 to R19, R132 to R20, R133 to R21, R134 to R22, R52 to R23, U13 to U4, U14 to U5
