File: Hardware/Design Files/rfsom-01/[12] - usb.kicad_sch (KiCad schematic)
At the start: 12 parts, among them U17 USB3320C-EZK, Y4 ECS-240-12-37B-CKY-TR

Commit message: aorus refresh;
Parts:
- U17: footprint Package_DFN_QFN:QFN-32-1EP_5x5mm_P0.5mm_EP3.1x3.1mm -> ICs:QFN-32-1EP_5x5mm_P0.5mm

Commit message: restructured project;
Parts:
- renumbered C202 to C164, C203 to C165, C204 to C166, C210 to C167, C211 to C168, R141 to R107, R142 to R108, R143 to R109, R144 to R110, R145 to R111, U17 to U11, Y4 to Y3
Changed lines of the file:
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@@
 		(dnp no)
 		(fields_autoplaced yes)
-		(property "Reference" "R145"
+		(property "Reference" "R111"
 			(at 219.71 78.7399 0)
 			(show_name no)
@@
 				)
 			)
+			(project "rfsom-01"
+				(path "/abe8d823-e11a-4177-8ce6-4f279cf45b05/8f56564b-be87-47cb-af1d-0a8f839d3522/5824b29f-0639-4332-9093-651d63d89232/f589e73c-86d1-4c53-a833-568491fb153e"
+					(reference "R111")
+					(unit 1)
+				)
+			)
 		)
 	)
@@
 		(dnp no)
 		(fields_autoplaced yes)
-		(property "Reference" "C204"
+		(property "Reference" "C166"
 			(at 129.54 29.2099 0)
 			(show_name no)
@@
 				)
 			)
+			(project "rfsom-01"
+				(path "/abe8d823-e11a-4177-8ce6-4f279cf45b05/8f56564b-be87-47cb-af1d-0a8f839d3522/5824b29f-0639-4332-9093-651d63d89232/f589e73c-86d1-4c53-a833-568491fb153e"
+					(reference "C166")
+					(unit 1)
+				)
+			)
 		)
 	)
@@
 		(dnp no)
 		(fields_autoplaced yes)
-		(property "Reference" "R142"
+		(property "Reference" "R108"
 			(at 185.42 104.1399 0)
 			(show_name no)
@@
 				)
 			)
+			(project "rfsom-01"
+				(path "/abe8d823-e11a-4177-8ce6-4f279cf45b05/8f56564b-be87-47cb-af1d-0a8f839d3522/5824b29f-0639-4332-9093-651d63d89232/f589e73c-86d1-4c53-a833-568491fb153e"
+					(reference "R108")
+					(unit 1)
+				)
+			)
 		)
 	)
@@
 		(dnp no)
 		(fields_autoplaced yes)
-		(property "Reference" "#PWR0267"
+		(property "Reference" "#PWR0205"
 			(at 116.84 95.25 0)
 			(hide yes)
@@
 				)
 			)
+			(project "rfsom-01"
+				(path "/abe8d823-e11a-4177-8ce6-4f279cf45b05/8f56564b-be87-47cb-af1d-0a8f839d3522/5824b29f-0639-4332-9093-651d63d89232/f589e73c-86d1-4c53-a833-568491fb153e"
+					(reference "#PWR0205")
+					(unit 1)
+				)
+			)
 		)
 	)
@@
 		(dnp no)
 		(fields_autoplaced yes)
-		(property "Reference" "C210"
+		(property "Reference" "C167"
 			(at 251.46 68.58 90)
 			(show_name no)
@@
 				)
 			)
+			(project "rfsom-01"
+				(path "/abe8d823-e11a-4177-8ce6-4f279cf45b05/8f56564b-be87-47cb-af1d-0a8f839d3522/5824b29f-0639-4332-9093-651d63d89232/f589e73c-86d1-4c53-a833-568491fb153e"
+					(reference "C167")
+					(unit 1)
+				)
+			)
 		)
 	)
@@
 		(dnp no)
 		(fields_autoplaced yes)
-		(property "Reference" "#PWR0247"
+		(property "Reference" "#PWR0212"
 			(at 227.33 96.52 0)
 			(hide yes)
@@
 				)
 			)
+			(project "rfsom-01"
+				(path "/abe8d823-e11a-4177-8ce6-4f279cf45b05/8f56564b-be87-47cb-af1d-0a8f839d3522/5824b29f-0639-4332-9093-651d63d89232/f589e73c-86d1-4c53-a833-568491fb153e"
+					(reference "#PWR0212")
+					(unit 1)
+				)
+			)
 		)
 	)
@@
 		(dnp no)
 		(fields_autoplaced yes)
-		(property "Reference" "#PWR0266"
+		(property "Reference" "#PWR0211"
 			(at 182.88 102.87 0)
 			(hide yes)
@@
 				)
 			)
+			(project "rfsom-01"
+				(path "/abe8d823-e11a-4177-8ce6-4f279cf45b05/8f56564b-be87-47cb-af1d-0a8f839d3522/5824b29f-0639-4332-9093-651d63d89232/f589e73c-86d1-4c53-a833-568491fb153e"
+					(reference "#PWR0211")
+					(unit 1)
+				)
+			)
 		)
 	)
@@
 		(dnp no)
 		(fields_autoplaced yes)
-		(property "Reference" "#PWR0262"
+		(property "Reference" "#PWR0210"
 			(at 177.8 38.1 0)
 			(hide yes)
@@
 				)
 			)
+			(project "rfsom-01"
+				(path "/abe8d823-e11a-4177-8ce6-4f279cf45b05/8f56564b-be87-47cb-af1d-0a8f839d3522/5824b29f-0639-4332-9093-651d63d89232/f589e73c-86d1-4c53-a833-568491fb153e"
+					(reference "#PWR0210")
+					(unit 1)
+				)
+			)
 		)
 	)
@@
 		(dnp no)
 		(fields_autoplaced yes)
-		(property "Reference" "C202"
+		(property "Reference" "C164"
 			(at 106.68 29.2099 0)
 			(show_name no)
@@
 				)
 			)
+			(project "rfsom-01"
+				(path "/abe8d823-e11a-4177-8ce6-4f279cf45b05/8f56564b-be87-47cb-af1d-0a8f839d3522/5824b29f-0639-4332-9093-651d63d89232/f589e73c-86d1-4c53-a833-568491fb153e"
+					(reference "C164")
+					(unit 1)
+				)
+			)
 		)
 	)
@@
 		(dnp no)
 		(fields_autoplaced yes)
-		(property "Reference" "#PWR0261"
+		(property "Reference" "#PWR0213"
 			(at 245.11 96.52 0)
 			(hide yes)
@@
 				)
 			)
+			(project "rfsom-01"
+				(path "/abe8d823-e11a-4177-8ce6-4f279cf45b05/8f56564b-be87-47cb-af1d-0a8f839d3522/5824b29f-0639-4332-9093-651d63d89232/f589e73c-86d1-4c53-a833-568491fb153e"
+					(reference "#PWR0213")
+					(unit 1)
+				)
+			)
 		)
 	)
@@
 		(dnp no)
 		(fields_autoplaced yes)
-		(property "Reference" "#PWR0264"
+		(property "Reference" "#PWR0206"
 			(at 125.73 27.94 0)
 			(hide yes)
@@
 				)
 			)
+			(project "rfsom-01"
+				(path "/abe8d823-e11a-4177-8ce6-4f279cf45b05/8f56564b-be87-47cb-af1d-0a8f839d3522/5824b29f-0639-4332-9093-651d63d89232/f589e73c-86d1-4c53-a833-568491fb153e"
+					(reference "#PWR0206")
+					(unit 1)
+				)
+			)
 		)
 	)
@@
 		(dnp no)
 		(fields_autoplaced yes)
-		(property "Reference" "U17"
+		(property "Reference" "U11"
 			(at 157.0833 102.87 0)
 			(show_name no)
@@
 				)
 			)
+			(project "rfsom-01"
+				(path "/abe8d823-e11a-4177-8ce6-4f279cf45b05/8f56564b-be87-47cb-af1d-0a8f839d3522/5824b29f-0639-4332-9093-651d63d89232/f589e73c-86d1-4c53-a833-568491fb153e"
+					(reference "U11")
+					(unit 1)
+				)
+			)
 		)
 	)
@@
 		(dnp no)
 		(fields_autoplaced yes)
-		(property "Reference" "#PWR0265"
+		(property "Reference" "#PWR0207"
 			(at 125.73 43.18 0)
 			(hide yes)
@@
 				)
 			)
+			(project "rfsom-01"
+				(path "/abe8d823-e11a-4177-8ce6-4f279cf45b05/8f56564b-be87-47cb-af1d-0a8f839d3522/5824b29f-0639-4332-9093-651d63d89232/f589e73c-86d1-4c53-a833-568491fb153e"
+					(reference "#PWR0207")
+					(unit 1)
+				)
+			)
 		)
 	)
@@
 		(dnp no)
 		(fields_autoplaced yes)
-		(property "Reference" "R141"
+		(property "Reference" "R107"
 			(at 133.35 99.0599 0)
 			(show_name no)
@@
 				)
 			)
+			(project "rfsom-01"
+				(path "/abe8d823-e11a-4177-8ce6-4f279cf45b05/8f56564b-be87-47cb-af1d-0a8f839d3522/5824b29f-0639-4332-9093-651d63d89232/f589e73c-86d1-4c53-a833-568491fb153e"
+					(reference "R107")
+					(unit 1)
+				)
+			)
 		)
 	)
@@
 		(dnp no)
 		(fields_autoplaced yes)
-		(property "Reference" "#PWR0312"
+		(property "Reference" "#PWR0215"
 			(at 264.16 85.09 0)
 			(hide yes)
@@
 				)
 			)
+			(project "rfsom-01"
+				(path "/abe8d823-e11a-4177-8ce6-4f279cf45b05/8f56564b-be87-47cb-af1d-0a8f839d3522/5824b29f-0639-4332-9093-651d63d89232/f589e73c-86d1-4c53-a833-568491fb153e"
+					(reference "#PWR0215")
+					(unit 1)
+				)
+			)
 		)
 	)
@@
 		(dnp no)
 		(fields_autoplaced yes)
-		(property "Reference" "#PWR0268"
+		(property "Reference" "#PWR0208"
 			(at 130.81 113.03 0)
 			(hide yes)
@@
 				)
 			)
+			(project "rfsom-01"
+				(path "/abe8d823-e11a-4177-8ce6-4f279cf45b05/8f56564b-be87-47cb-af1d-0a8f839d3522/5824b29f-0639-4332-9093-651d63d89232/f589e73c-86d1-4c53-a833-568491fb153e"
+					(reference "#PWR0208")
+					(unit 1)
+				)
+			)
 		)
 	)
@@
 		(in_pos_files yes)
 		(dnp yes)
-		(property "Reference" "R143"
+		(property "Reference" "R109"
 			(at 210.566 76.2 90)
 			(show_name no)
@@
 				)
 			)
+			(project "rfsom-01"
+				(path "/abe8d823-e11a-4177-8ce6-4f279cf45b05/8f56564b-be87-47cb-af1d-0a8f839d3522/5824b29f-0639-4332-9093-651d63d89232/f589e73c-86d1-4c53-a833-568491fb153e"
+					(reference "R109")
+					(unit 1)
+				)
+			)
 		)
 	)
@@
 		(dnp no)
 		(fields_autoplaced yes)
-		(property "Reference" "C203"
+		(property "Reference" "C165"
 			(at 118.11 29.2099 0)
 			(show_name no)
@@
 				)
 			)
+			(project "rfsom-01"
+				(path "/abe8d823-e11a-4177-8ce6-4f279cf45b05/8f56564b-be87-47cb-af1d-0a8f839d3522/5824b29f-0639-4332-9093-651d63d89232/f589e73c-86d1-4c53-a833-568491fb153e"
+					(reference "C165")
+					(unit 1)
+				)
+			)
 		)
 	)
@@
 		(dnp no)
 		(fields_autoplaced yes)
-		(property "Reference" "#PWR0263"
+		(property "Reference" "#PWR0209"
 			(at 149.86 38.1 0)
 			(hide yes)
@@
 				)
 			)
+			(project "rfsom-01"
+				(path "/abe8d823-e11a-4177-8ce6-4f279cf45b05/8f56564b-be87-47cb-af1d-0a8f839d3522/5824b29f-0639-4332-9093-651d63d89232/f589e73c-86d1-4c53-a833-568491fb153e"
+					(reference "#PWR0209")
+					(unit 1)
+				)
+			)
 		)
 	)
@@
 		(dnp no)
 		(fields_autoplaced yes)
-		(property "Reference" "#PWR0311"
+		(property "Reference" "#PWR0214"
 			(at 264.16 74.93 0)
 			(hide yes)
@@
 				)
 			)
+			(project "rfsom-01"
+				(path "/abe8d823-e11a-4177-8ce6-4f279cf45b05/8f56564b-be87-47cb-af1d-0a8f839d3522/5824b29f-0639-4332-9093-651d63d89232/f589e73c-86d1-4c53-a833-568491fb153e"
+					(reference "#PWR0214")
+					(unit 1)
+				)
+			)
 		)
 	)
@@
 		(dnp no)
 		(fields_autoplaced yes)
-		(property "Reference" "C211"
+		(property "Reference" "C168"
 			(at 251.46 78.74 90)
 			(show_name no)
@@
 				)
 			)
+			(project "rfsom-01"
+				(path "/abe8d823-e11a-4177-8ce6-4f279cf45b05/8f56564b-be87-47cb-af1d-0a8f839d3522/5824b29f-0639-4332-9093-651d63d89232/f589e73c-86d1-4c53-a833-568491fb153e"
+					(reference "C168")
+					(unit 1)
+				)
+			)
 		)
 	)
@@
 		(in_pos_files yes)
 		(dnp yes)
-		(property "Reference" "R144"
+		(property "Reference" "R110"
 			(at 210.566 81.28 90)
 			(show_name no)
@@
 				)
 			)
+			(project "rfsom-01"
+				(path "/abe8d823-e11a-4177-8ce6-4f279cf45b05/8f56564b-be87-47cb-af1d-0a8f839d3522/5824b29f-0639-4332-9093-651d63d89232/f589e73c-86d1-4c53-a833-568491fb153e"
+					(reference "R110")
+					(unit 1)
+				)
+			)
 		)
 	)
@@
 		(in_pos_files yes)
 		(dnp no)
-		(property "Reference" "Y4"
+		(property "Reference" "Y3"
 			(at 235.204 67.818 90)
 			(show_name no)
@@
 					(unit 1)
 				)
+			)
+			(project "rfsom-01"
+				(path "/abe8d823-e11a-4177-8ce6-4f279cf45b05/8f56564b-be87-47cb-af1d-0a8f839d3522/5824b29f-0639-4332-9093-651d63d89232/f589e73c-86d1-4c53-a833-568491fb153e"
+					(reference "Y3")
+					(unit 1)
+				)
