File: Hardware/Design Files/rfsom-01/[13] - eth-phy.kicad_sch (KiCad schematic)
At the start: 50 parts, among them U6 KSZ9131RNXI-TR, Y3 ECS-2033-250-BN

Commit message: restructured project;
Parts:
- renumbered C205 to C175, C206 to C176, C185 to C177, C207 to C178, C208 to C179, C209 to C180, C16 to C181, C17 to C182, C18 to C183, C19 to C184, C20 to C185, C21 to C186, C22 to C187, C23 to C188, C24 to C189, C25 to C190, C26 to C191, C27 to C192, C28 to C193, C29 to C194, C30 to C195, C31 to C196, C32 to C197, FB5 to FB10, FB6 to FB11, FB7 to FB12, FB2 to FB7, FB3 to FB8, FB4 to FB9, R13 to R115, R14 to R116, R15 to R117, R16 to R118, R17 to R119, R18 to R120, R19 to R121, R20 to R122, R21 to R123, R22 to R124, R23 to R125, R27 to R126, R28 to R127, R29 to R128, R30 to R129, R31 to R130, R32 to R131, R33 to R132, R34 to R133, U6 to U13, Y3 to Y4
