File: Hardware/Design Files/rfsom-01/[14] - ftdi.kicad_sch (KiCad schematic)
At the start: 39 parts, among them J2 2216100001, U16 93LC56BT-I/OT, U4 FT232HQ-REEL, Y2 ABM10-166-12.000MHZ-T3

Commit message: restructured project;
Parts:
- renumbered C199 to C1, C39 to C10, C40 to C11, C41 to C12, C42 to C13, C43 to C14, C44 to C15, C45 to C16, C200 to C2, C201 to C3, C33 to C4, C34 to C5, C35 to C6, C36 to C7, C37 to C8, C38 to C9, FB12 to FB2, FB8 to FB3, FB9 to FB4, R137 to R1, R38 to R10, R39 to R11, R40 to R12, R41 to R13, R6 to R2, R138 to R3, R139 to R4, R7 to R5, R140 to R6, R35 to R7, R37 to R8, R36 to R9, U16 to U1, U4 to U2, Y2 to Y1
