File: Hardware/Design Files/rfsom-01/[15] - mezzanine.kicad_sch (KiCad schematic)
At the start: 2 parts, among them J10 SEAM-40-02.0-L-04-2-A-K-TR, J3 SEAM-40-02.0-L-04-2-A-K-TR

Commit message: restructured project;
Parts:
- renumbered J3 to J7, J10 to J8
Changed lines of the file:
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@@
 		(dnp no)
 		(fields_autoplaced yes)
-		(property "Reference" "J10"
+		(property "Reference" "J8"
 			(at 229.87 87.63 0)
 			(show_name no)
@@
 				)
 			)
+			(project "rfsom-01"
+				(path "/abe8d823-e11a-4177-8ce6-4f279cf45b05/8f56564b-be87-47cb-af1d-0a8f839d3522/aa769d64-0dd0-48a6-88b3-65c6d6ecbe65"
+					(reference "J8")
+					(unit 3)
+				)
+			)
 		)
 	)
@@
 		(dnp no)
 		(fields_autoplaced yes)
-		(property "Reference" "J3"
+		(property "Reference" "J7"
 			(at 59.69 125.73 0)
 			(show_name no)
@@
 				)
 			)
+			(project "rfsom-01"
+				(path "/abe8d823-e11a-4177-8ce6-4f279cf45b05/8f56564b-be87-47cb-af1d-0a8f839d3522/aa769d64-0dd0-48a6-88b3-65c6d6ecbe65"
+					(reference "J7")
+					(unit 2)
+				)
+			)
 		)
 	)
@@
 		(dnp no)
 		(fields_autoplaced yes)
-		(property "Reference" "J10"
+		(property "Reference" "J8"
 			(at 194.31 87.63 0)
 			(show_name no)
@@
 				)
 			)
+			(project "rfsom-01"
+				(path "/abe8d823-e11a-4177-8ce6-4f279cf45b05/8f56564b-be87-47cb-af1d-0a8f839d3522/aa769d64-0dd0-48a6-88b3-65c6d6ecbe65"
+					(reference "J8")
+					(unit 2)
+				)
+			)
 		)
 	)
@@
 		(dnp no)
 		(fields_autoplaced yes)
-		(property "Reference" "#PWR07"
+		(property "Reference" "#PWR0344"
 			(at 243.84 43.18 0)
 			(hide yes)
@@
 				)
 			)
+			(project "rfsom-01"
+				(path "/abe8d823-e11a-4177-8ce6-4f279cf45b05/8f56564b-be87-47cb-af1d-0a8f839d3522/aa769d64-0dd0-48a6-88b3-65c6d6ecbe65"
+					(reference "#PWR0344")
+					(unit 1)
+				)
+			)
 		)
 	)
@@
 		(dnp no)
 		(fields_autoplaced yes)
-		(property "Reference" "J3"
+		(property "Reference" "J7"
 			(at 132.08 125.73 0)
 			(show_name no)
@@
 				)
 			)
+			(project "rfsom-01"
+				(path "/abe8d823-e11a-4177-8ce6-4f279cf45b05/8f56564b-be87-47cb-af1d-0a8f839d3522/aa769d64-0dd0-48a6-88b3-65c6d6ecbe65"
+					(reference "J7")
+					(unit 4)
+				)
+			)
 		)
 	)
@@
 		(dnp no)
 		(fields_autoplaced yes)
-		(property "Reference" "J3"
+		(property "Reference" "J7"
 			(at 95.25 125.73 0)
 			(show_name no)
@@
 				)
 			)
+			(project "rfsom-01"
+				(path "/abe8d823-e11a-4177-8ce6-4f279cf45b05/8f56564b-be87-47cb-af1d-0a8f839d3522/aa769d64-0dd0-48a6-88b3-65c6d6ecbe65"
+					(reference "J7")
+					(unit 3)
+				)
+			)
 		)
 	)
@@
 		(dnp no)
 		(fields_autoplaced yes)
-		(property "Reference" "J10"
+		(property "Reference" "J8"
 			(at 158.75 87.63 0)
 			(show_name no)
@@
 				)
 			)
+			(project "rfsom-01"
+				(path "/abe8d823-e11a-4177-8ce6-4f279cf45b05/8f56564b-be87-47cb-af1d-0a8f839d3522/aa769d64-0dd0-48a6-88b3-65c6d6ecbe65"
+					(reference "J8")
+					(unit 1)
+				)
+			)
 		)
 	)
@@
 		(dnp no)
 		(fields_autoplaced yes)
-		(property "Reference" "J10"
+		(property "Reference" "J8"
 			(at 266.7 87.63 0)
 			(show_name no)
@@
 				)
 			)
+			(project "rfsom-01"
+				(path "/abe8d823-e11a-4177-8ce6-4f279cf45b05/8f56564b-be87-47cb-af1d-0a8f839d3522/aa769d64-0dd0-48a6-88b3-65c6d6ecbe65"
+					(reference "J8")
+					(unit 4)
+				)
+			)
 		)
 	)
@@
 		(dnp no)
 		(fields_autoplaced yes)
-		(property "Reference" "J3"
+		(property "Reference" "J7"
 			(at 24.13 125.73 0)
 			(show_name no)
@@
 					(unit 1)
 				)
+			)
+			(project "rfsom-01"
+				(path "/abe8d823-e11a-4177-8ce6-4f279cf45b05/8f56564b-be87-47cb-af1d-0a8f839d3522/aa769d64-0dd0-48a6-88b3-65c6d6ecbe65"
+					(reference "J7")
+					(unit 1)
+				)
